File: HALSER.kicad_pcb (KiCad board)
At the start: 4 copper layers, 89 x 58 mm, 227 parts, among them J1103 Conn_01x02, J1104 Conn_01x02, J1105 Conn_01x02, J1106 Conn_01x02, J1201 Conn_01x02, J201 GPIO, J203 Conn_01x01, J302 Conn_01x02, J401 USB_B_Micro, J602 Conn_02x04_Odd_Even, J604 Conn_01x02, J605 Conn_01x02, J606 Conn_01x02, J607 Conn_01x02, J702 Conn_01x04, J801 Conn_01x03, J802 Conn_01x04, Q401 S8050, Q402 S8050, Q601 S9015, Q602 S9015, Q603 S9015, Q604 S9015, SW501 SW_Push, SW502 SW_Push, U1101 74LVC1G17, U1102 74LVC1G17, U1103 74LVC1G17, U1104 74LVC1G17, U1201 π140U30, U1202 ISO1540, U1203 XC6206P332MR, U201 ESP32-WROOM-32E-N16, U202 XL1509-3.3, U401 CH340C, U501 SN65HVD230DR, U601 LMV324, U602 ADS1115IDGS

Commit message: WIP wiring
Parts:
- removed C1101, C1102, C1103, C1112: 3.3nF, Capacitor_SMD:C_0402_1005Metric
- removed C1104, C1105, C1106, C1107: 220pF, Resistor_SMD:R_0402_1005Metric
- removed C1113, C1114, C1115, C1116, C1205, C1206, C606, C607, C608, C609, C610, C624: 100nF, Capacitor_SMD:C_0402_1005Metric
- removed the C304 at (125.8, 112.4)
- removed the C403 at (169.3, 94.7)
- removed the C404 at (169.3, 96.7)
- removed the C501 at (166.8, 102.2)
- removed the C502 at (170.3, 108.4)
- removed C601, C604, C612, C614: 33pF/50V, Capacitor_SMD:C_0603_1608Metric
- removed C603, C605, C613, C615: 33pF, Capacitor_SMD:C_0402_1005Metric
- removed C611: 68nF, Capacitor_SMD:C_0603_1608Metric
- removed C620, C621, C622, C623: 10nF, Capacitor_SMD:C_0402_1005Metric
- removed C710, C711, C712, C714: 10uF/50V, Capacitor_SMD:C_1206_3216Metric
- removed C713: 4.7nF/50V, Capacitor_SMD:C_0402_1005Metric
- removed C715: 1uF/50V, Capacitor_SMD:C_0805_2012Metric
- removed C716: 4.7uF/50V, Capacitor_SMD:C_1206_3216Metric
- removed the C901 at (165.2, 92.0)
- removed D1101, D1102: BAT54A, Package_TO_SOT_SMD:SOT-323_SC-70
- removed D1103, D1104, D1105, D1113, D603, D604, D605, D611: BAT54S, Package_TO_SOT_SMD:SOT-323_SC-70
- removed the D501 at (175.2, 104.9)
- removed the D502 at (175.2, 102.8)
- removed the D701 at (124.8, 108.3)
- removed the D801 at (110.8, 99.2)
- removed FB601, FB602, FB603, FB604: GZ2012D101TF, Inductor_SMD:L_0805_2012Metric
- removed FB704: GZ2012D601TF, Inductor_SMD:L_0805_2012Metric
- removed J1103, J1104, J1105, J1106, J604, J605, J606, J607: Conn_01x02, Connector_Phoenix_MC:PhoenixContact_MCV_1,5_2-G-3.81_1x02_P3.81mm_Vertical
- removed J201: GPIO, Connector_PinHeader_2.54mm:PinHeader_2x10_P2.54mm_Vertical
- removed J203: Conn_01x01, TestPoint:TestPoint_Pad_D2.0mm
- removed J302: Conn_01x02, Connector_PinHeader_2.54mm:PinHeader_1x02_P2.54mm_Vertical
- removed the J401 at (174.5, 98.8)
- removed J602: Conn_02x04_Odd_Even, Connector_PinHeader_2.54mm:PinHeader_2x04_P2.54mm_Vertical
- removed JP1101, JP1102, JP1103, JP1104, JP1105, JP1106, JP1107, JP1108, JP1109, JP1110, JP1111, JP1112, JP601: SolderJumper_2_Open, HALMET:SolderJumper-2_P1.3mm_Open_TrianglePad_Narrow
- removed JP602, JP604, JP605: Open, Jumper:SolderJumper-2_P1.3mm_Open_Pad1.0x1.5mm
- removed JP603: Bridged, Jumper:SolderJumper-2_P1.3mm_Bridged2Bar_RoundedPad1.0x1.5mm
- removed Q401, Q402: S8050, Package_TO_SOT_SMD:SOT-23
- removed Q601, Q602, Q603, Q604: S9015, Package_TO_SOT_SMD:SOT-323_SC-70
- removed R1101, R1102, R1104, R1105, R613, R614, R616, R618: 20k, Resistor_SMD:R_0603_1608Metric
- removed R1106, R1107, R1108, R1109: 100k, Resistor_SMD:R_0402_1005Metric
- removed R1202, R1203: 2k, Resistor_SMD:R_0402_1005Metric
- removed the R401 at (161.2, 92.0)
- removed the R402 at (163.2, 92.0)
- removed the R501 at (172.6, 104.9)
- removed the R502 at (172.6, 103.4)
- removed R601, R602: 240R, Resistor_SMD:R_0805_2012Metric
- removed R603, R604, R605, R606, R611: 1k, Resistor_SMD:R_0402_1005Metric
- removed R607, R608, R609, R610: 30, Resistor_SMD:R_0603_1608Metric
- removed R612: 10k, Resistor_SMD:R_0402_1005Metric
- removed R615, R617, R619, R621: 2.2k, Resistor_SMD:R_0402_1005Metric
- removed the REF** at (167.2, 74.9)
- removed SW501, SW502: SW_Push, Button_Switch_SMD:SW_SPST_TL3342
- removed U1101, U1102, U1103, U1104: 74LVC1G17, Package_TO_SOT_SMD:SOT-353_SC-70-5
- removed U1201: π140U30, Package_SO:SOIC-16_4.55x10.3mm_P1.27mm
- removed U1202: ISO1540, Package_SO:SOIC-8_3.9x4.9mm_P1.27mm
- removed the U201 at (162.3, 76.1)
- removed U202: XL1509-3.3, Package_SO:SOP-8_3.9x4.9mm_P1.27mm
- removed U401: CH340C, Package_SO:SOIC-16_3.9x9.9mm_P1.27mm
- removed U601: LMV324, Package_SO:SOIC-14_3.9x8.7mm_P1.27mm
- removed U602: ADS1115IDGS, Package_SO:TSSOP-10_3x3mm_P0.5mm
- added C1001: 100nF, PCM_Capacitor_SMD_AKL:C_0402_1005Metric, F.Cu at (99.4, 61.2)
- added C1002: 100nF, PCM_Capacitor_SMD_AKL:C_0402_1005Metric, F.Cu at (99.4, 108.4)
- added C1003: 100nF, PCM_Capacitor_SMD_AKL:C_0402_1005Metric, F.Cu at (114.8, 67.6)
- added C1004: 100nF, PCM_Capacitor_SMD_AKL:C_0402_1005Metric, F.Cu at (124.4, 68.6)
- added C1005: 100nF, PCM_Capacitor_SMD_AKL:C_0402_1005Metric, F.Cu at (116.2, 103.5)
- added C1006: 100nF, PCM_Capacitor_SMD_AKL:C_0402_1005Metric, F.Cu at (124.4, 66.2)
- added C1007: 100nF, PCM_Capacitor_SMD_AKL:C_0402_1005Metric, F.Cu at (124.4, 67.4)
- added C1008: 100pF, PCM_Capacitor_SMD_AKL:C_0603_1608Metric, F.Cu at (92.2, 67.2)
- added C1009: 100pF, PCM_Capacitor_SMD_AKL:C_0603_1608Metric, F.Cu at (98.4, 102.3)
- added C1010: 100pF, PCM_Capacitor_SMD_AKL:C_0603_1608Metric, F.Cu at (92.2, 69.0)
- added C1011: 100pF, PCM_Capacitor_SMD_AKL:C_0603_1608Metric, F.Cu at (100.2, 102.3)
- added C1012: 100pF, PCM_Capacitor_SMD_AKL:C_0603_1608Metric, F.Cu at (117.4, 101.2)
- added C1013: 100pF, PCM_Capacitor_SMD_AKL:C_0603_1608Metric, F.Cu at (106.8, 98.9)
- added C1014: 100pF, PCM_Capacitor_SMD_AKL:C_0603_1608Metric, F.Cu at (120.1, 92.0)
- added C1015: 100pF, PCM_Capacitor_SMD_AKL:C_0603_1608Metric, F.Cu at (106.8, 93.0)
- added C1016: 150pF/50V, PCM_Capacitor_SMD_AKL:C_0603_1608Metric, F.Cu at (110.0, 68.8)
- added C1017: 150pF/50V, PCM_Capacitor_SMD_AKL:C_0603_1608Metric, F.Cu at (120.8, 70.3)
- added C1018: 150pF/50V, PCM_Capacitor_SMD_AKL:C_0603_1608Metric, F.Cu at (106.6, 71.3)
- added C1019: 150pF/50V, PCM_Capacitor_SMD_AKL:C_0603_1608Metric, F.Cu at (120.5, 74.3)
- added C201: 100pF, PCM_Capacitor_SMD_AKL:C_0603_1608Metric, F.Cu at (146.4, 91.8)
- added C202: 100pF, PCM_Capacitor_SMD_AKL:C_0603_1608Metric, F.Cu at (142.2, 91.8)
- added C301: 100nF/50V, PCM_Capacitor_SMD_AKL:C_0603_1608Metric, F.Cu at (171.9, 97.7)
- added C302: 100nF/50V, PCM_Capacitor_SMD_AKL:C_0603_1608Metric, F.Cu at (171.9, 103.9)
- added C305: 100nF, PCM_Capacitor_SMD_AKL:C_0402_1005Metric, F.Cu at (170.8, 66.9)
- added C701: 10uF/50V, PCM_Capacitor_SMD_AKL:C_1206_3216Metric, F.Cu at (140.7, 111.1)
- added C702: 4.7uF/50V, PCM_Capacitor_SMD_AKL:C_0805_2012Metric, F.Cu at (136.1, 111.1)
- added C703: 10uF/50V, PCM_Capacitor_SMD_AKL:C_1206_3216Metric, F.Cu at (132.9, 109.2)
- added C704: 10uF/50V, PCM_Capacitor_SMD_AKL:C_1206_3216Metric, F.Cu at (135.6, 107.4)
- added C705: 10uF/50V, PCM_Capacitor_SMD_AKL:C_1206_3216Metric, F.Cu at (127.6, 112.0)
- added C706: 100nF/50V, PCM_Capacitor_SMD_AKL:C_0603_1608Metric, F.Cu at (130.8, 109.7)
- added D1003: SM712_SOT23, PCM_Package_TO_SOT_SMD_AKL:SOT-23, F.Cu at (92.2, 71.9)
- added D1004: SM712_SOT23, PCM_Package_TO_SOT_SMD_AKL:SOT-23, F.Cu at (92.1, 102.6)
- added D1005: SMAJ16CA, PCM_Diode_SMD_AKL:D_SMA_TVS, F.Cu at (92.1, 77.8)
- added D1006: SMAJ16CA, PCM_Diode_SMD_AKL:D_SMA_TVS, F.Cu at (92.1, 97.0)
- added D1007: ESD5451N, PCM_Diode_SMD_AKL:D_0402_1005Metric, F.Cu at (119.6, 90.4)
- added D1008: PESD15VS2UT, PCM_Package_TO_SOT_SMD_AKL:SOT-23, F.Cu at (120.5, 77.1)
- added D1009: ESD5451N, PCM_Diode_SMD_AKL:D_0402_1005Metric, F.Cu at (106.4, 91.4)
- added D201: SM24CANB, PCM_Package_TO_SOT_SMD_AKL:SOT-23, F.Cu at (144.3, 88.1)
- added D301: RED LED, PCM_LED_SMD_AKL:LED_0603_1608Metric, F.Cu at (165.8, 60.9)
- added D302: GREEN LED, PCM_LED_SMD_AKL:LED_0603_1608Metric, F.Cu at (142.0, 77.1)
- added D303: GREEN LED, PCM_LED_SMD_AKL:LED_0603_1608Metric, F.Cu at (146.6, 77.1)
- added F1001: nSMD005/60V, PCM_Fuse_AKL:Fuse_1206_3216Metric, F.Cu at (92.7, 83.0)
- added F1002: nSMD005/60V, PCM_Fuse_AKL:Fuse_1206_3216Metric, F.Cu at (92.7, 85.9)
- added F1003: nSMD005/60V, PCM_Fuse_AKL:Fuse_1206_3216Metric, F.Cu at (92.7, 88.9)
- added F1004: nSMD005/60V, PCM_Fuse_AKL:Fuse_1206_3216Metric, F.Cu at (92.7, 91.8)
- added FB1001: GZ2012D601TF, PCM_Ferrite_SMD_AKL:Ferrite_0805_2012Metric, F.Cu at (119.5, 95.0)
- added FB1002: GZ2012D601TF, PCM_Ferrite_SMD_AKL:Ferrite_0805_2012Metric, F.Cu at (106.5, 96.0)
- added FB1003: GZ2012D601TF, PCM_Ferrite_SMD_AKL:Ferrite_0805_2012Metric, F.Cu at (109.5, 70.8)
- added FB1004: GZ2012D601TF, PCM_Ferrite_SMD_AKL:Ferrite_0805_2012Metric, F.Cu at (120.5, 72.3)
- added FL1001: PCAQ2012B-201T030, HALSER:L_CommonModeChoke_PCAQ2012B, F.Cu at (95.4, 68.9)
- added FL1002: PCAQ2012B-201T030, HALSER:L_CommonModeChoke_PCAQ2012B, F.Cu at (95.7, 101.9)
- added FL201: PCAQ2012B-201T030, HALSER:L_CommonModeChoke_PCAQ2012B, F.Cu at (144.3, 91.8)
- added G603: WEEE-logo, Symbol:WEEE-Logo_5.6x8mm_SilkScreen, F.Cu at (276.0, 122.8)
- added H603: MountingHole, MountingHole:MountingHole_3.2mm_M3_ISO7380, F.Cu at (156.5, 63.0)
- added H604: MountingHole, MountingHole:MountingHole_3.2mm_M3_ISO7380, F.Cu at (156.5, 109.0)
- added J1001: RX Sel Header, Connector_PinHeader_2.54mm:PinHeader_2x03_P2.54mm_Vertical, F.Cu at (103.9, 66.9)
- added J1002: RS485 RX Socket, Connector_Phoenix_MC:PhoenixContact_MCV_1,5_3-G-3.81_1x03_P3.81mm_Vertical, F.Cu at (101.8, 82.8)
- added J1003: RS485 TX Socket, Connector_Phoenix_MC:PhoenixContact_MCV_1,5_3-G-3.81_1x03_P3.81mm_Vertical, F.Cu at (101.8, 96.8)
- added J1004: RS-232 Socket, Connector_Phoenix_MC:PhoenixContact_MCV_1,5_3-G-3.81_1x03_P3.81mm_Vertical, F.Cu at (114.8, 82.8)
- added J1005: UART Socket, Connector_Phoenix_MC:PhoenixContact_MCV_1,5_3-G-3.81_1x03_P3.81mm_Vertical, F.Cu at (114.8, 96.8)
- added J301: GPIO, Connector_PinHeader_2.54mm:PinHeader_2x10_P2.54mm_Vertical, F.Cu at (153.3, 74.6)
- added J701: CAN Socket, Connector_Phoenix_MC:PhoenixContact_MCV_1,5_4-G-3.81_1x04_P3.81mm_Vertical, F.Cu at (146.8, 100.0)
- added LED301: SK68XX-MINI-HS, PCM_LED_SMD_AKL:LED_SK6812MINI_PLCC4_3.5x3.5mm_P1.75mm, F.Cu at (175.3, 97.7)
- added R1003: 470R, PCM_Resistor_SMD_AKL:R_0402_1005Metric, F.Cu at (117.5, 103.5)
- added R1004: 470R, PCM_Resistor_SMD_AKL:R_0402_1005Metric, F.Cu at (110.9, 101.7)
- added R1005: 10R, PCM_Resistor_SMD_AKL:R_0402_1005Metric, F.Cu at (94.8, 66.2)
- added R1006: 10R, PCM_Resistor_SMD_AKL:R_0402_1005Metric, F.Cu at (96.0, 66.2)
- added R1007: 10R, PCM_Resistor_SMD_AKL:R_0402_1005Metric, F.Cu at (102.9, 102.8)
- added R1008: 10R, PCM_Resistor_SMD_AKL:R_0402_1005Metric, F.Cu at (101.7, 102.8)
- added R1009: 51R, PCM_Resistor_SMD_AKL:R_0603_1608Metric, F.Cu at (110.0, 67.0)
- added R1010: 51R, PCM_Resistor_SMD_AKL:R_0603_1608Metric, F.Cu at (117.5, 70.3)
- added R303: 2k, PCM_Resistor_SMD_AKL:R_0402_1005Metric, F.Cu at (163.9, 61.5)
- added R304: 1.5k, PCM_Resistor_SMD_AKL:R_0402_1005Metric, F.Cu at (141.5, 79.0)
- added R305: 1.5k, PCM_Resistor_SMD_AKL:R_0402_1005Metric, F.Cu at (147.1, 79.0)
- added R306: 0R, PCM_Resistor_SMD_AKL:R_0603_1608Metric, F.Cu at (175.2, 93.7)
- added R701: 0.1R, PCM_Resistor_SMD_AKL:R_0603_1608Metric, F.Cu at (132.6, 112.6)
- added R702: 75k, PCM_Resistor_SMD_AKL:R_0402_1005Metric, F.Cu at (124.6, 110.1)
- added R801: 5.1k, PCM_Resistor_SMD_AKL:R_0402_1005Metric, F.Cu at (170.4, 86.4)
- added R802: 5.1k, PCM_Resistor_SMD_AKL:R_0402_1005Metric, F.Cu at (170.4, 88.6)
- added SW301: SW_Push, Button_Switch_SMD:SW_SPST_TL3342, F.Cu at (166.7, 97.7)
- added SW302: SW_Push, Button_Switch_SMD:SW_SPST_TL3342, F.Cu at (166.7, 103.9)
- added U1001: SN75176BDR, PCM_Package_SO_AKL:SOIC-8_3.9x4.9mm_P1.27mm, F.Cu at (103.9, 61.2)
- added U1002: 74LVC2G17, PCM_Package_TO_SOT_SMD_AKL:SOT-23-6, F.Cu at (113.6, 102.7)
- added U1003: SP3232EEY-L/TR, PCM_Package_SO_AKL:TSSOP-16_4.4x5mm_P0.65mm, F.Cu at (119.3, 65.7)
- added U1004: SN75176BDR, PCM_Package_SO_AKL:SOIC-8_3.9x4.9mm_P1.27mm, F.Cu at (103.9, 108.4)
- added U301: ESP32-C3-MINI-1, PCM_Espressif:ESP32-C3-MINI-1, F.Cu at (170.7, 74.4)
- added U701: LMR54410DBVR, PCM_Package_TO_SOT_SMD_AKL:SOT-23-6, F.Cu at (127.8, 108.7)
- added U901: π122U31, PCM_Package_SO_AKL:SOIC-8_3.9x4.9mm_P1.27mm, F.Cu at (129.4, 73.7)
- C203: renamed from C602; footprint Capacitor_SMD:C_0402_1005Metric -> PCM_Capacitor_SMD_AKL:C_0402_1005Metric
- C303: renamed from C203; footprint Capacitor_SMD:C_0402_1005Metric -> PCM_Capacitor_SMD_AKL:C_0402_1005Metric
- C304: renamed from C202; value 22uF -> 10uF/25V; footprint Capacitor_SMD:C_0603_1608Metric -> PCM_Capacitor_SMD_AKL:C_0805_2012Metric
- C401: renamed from C704; footprint Capacitor_SMD:C_1206_3216Metric -> PCM_Capacitor_SMD_AKL:C_1206_3216Metric
- C402: renamed from C705; footprint Capacitor_SMD:C_0603_1608Metric -> PCM_Capacitor_SMD_AKL:C_0603_1608Metric
- C403: renamed from C706; footprint Capacitor_SMD:C_0603_1608Metric -> PCM_Capacitor_SMD_AKL:C_0603_1608Metric
- C404: renamed from C701; footprint Capacitor_SMD:C_0402_1005Metric -> PCM_Capacitor_SMD_AKL:C_0603_1608Metric
- C405: renamed from C702; footprint Capacitor_SMD:C_0402_1005Metric -> PCM_Capacitor_SMD_AKL:C_0402_1005Metric
- C406: renamed from C703; footprint Capacitor_SMD:C_0402_1005Metric -> PCM_Capacitor_SMD_AKL:C_0402_1005Metric
- C501: renamed from C803; footprint Capacitor_SMD:C_1206_3216Metric -> PCM_Capacitor_SMD_AKL:C_1206_3216Metric
- C502: renamed from C802; footprint Capacitor_SMD:C_0603_1608Metric -> PCM_Capacitor_SMD_AKL:C_0603_1608Metric
- C503: renamed from C801; footprint Capacitor_SMD:C_0402_1005Metric -> PCM_Capacitor_SMD_AKL:C_0603_1608Metric
- C707: value 10uF/50V -> 100nF/16V; footprint Capacitor_SMD:C_1206_3216Metric -> PCM_Capacitor_SMD_AKL:C_0402_1005Metric
- C708, C709: value 10uF/50V -> 47uF/6.3V; footprint Capacitor_SMD:C_1206_3216Metric -> PCM_Capacitor_SMD_AKL:C_0805_2012Metric
- C801: renamed from C503; footprint Capacitor_SMD:C_0805_2012Metric -> PCM_Capacitor_SMD_AKL:C_0603_1608Metric
- C802: renamed from C402; footprint Capacitor_SMD:C_0603_1608Metric -> PCM_Capacitor_SMD_AKL:C_0603_1608Metric
- C901: renamed from C1201; footprint Capacitor_SMD:C_0402_1005Metric -> PCM_Capacitor_SMD_AKL:C_0603_1608Metric
- C902: renamed from C1207; footprint Capacitor_SMD:C_0402_1005Metric -> PCM_Capacitor_SMD_AKL:C_0402_1005Metric
- C903: renamed from C1208; footprint Capacitor_SMD:C_0402_1005Metric -> PCM_Capacitor_SMD_AKL:C_0603_1608Metric
- C904: renamed from C1209; footprint HALMET:C_1808_4520Metric -> HALSER:C_1808_4520Metric
- C905: renamed from C1210; footprint Capacitor_SMD:C_0402_1005Metric -> PCM_Capacitor_SMD_AKL:C_0603_1608Metric
- C906: renamed from C1204; footprint Capacitor_SMD:C_0402_1005Metric -> PCM_Capacitor_SMD_AKL:C_0402_1005Metric
- C907: renamed from C1202; footprint Capacitor_SMD:C_0402_1005Metric -> PCM_Capacitor_SMD_AKL:C_0603_1608Metric
- C908: renamed from C1203; footprint Capacitor_SMD:C_0603_1608Metric -> PCM_Capacitor_SMD_AKL:C_0603_1608Metric
- D1001, D1002: footprint LED_SMD:LED_0603_1608Metric -> PCM_LED_SMD_AKL:LED_0603_1608Metric
- D401, D402, D403: footprint Diode_SMD:D_0402_1005Metric -> PCM_Diode_SMD_AKL:D_0402_1005Metric
- D501: renamed from D503; footprint Diode_SMD:D_0402_1005Metric -> PCM_Diode_SMD_AKL:D_0402_1005Metric
- D502: renamed from D504; footprint Diode_SMD:D_0402_1005Metric -> PCM_Diode_SMD_AKL:D_0402_1005Metric
- D701: renamed from D201; footprint Diode_SMD:D_SOD-123 -> PCM_Diode_SMD_AKL:D_SOD-123
- D702: renamed from D301; footprint Diode_SMD:D_SMB -> PCM_Diode_SMD_AKL:D_SMB_TVS
- D703: renamed from D303; footprint Diode_SMD:D_SOD-123 -> PCM_Diode_SMD_AKL:D_SOD-123
- D801: renamed from D903; footprint Diode_SMD:D_0402_1005Metric -> PCM_Diode_SMD_AKL:D_0402_1005Metric
- D802: renamed from D904; footprint Diode_SMD:D_0402_1005Metric -> PCM_Diode_SMD_AKL:D_0402_1005Metric
- D803: renamed from D905; footprint Diode_SMD:D_0402_1005Metric -> PCM_Diode_SMD_AKL:D_0402_1005Metric
- F701: renamed from F301; footprint Fuse:Fuse_1812_4532Metric -> PCM_Fuse_AKL:Fuse_1812_4532Metric
- F801: renamed from F401; footprint Fuse:Fuse_1206_3216Metric -> PCM_Fuse_AKL:Fuse_1206_3216Metric
- FB401: renamed from FB701; footprint Inductor_SMD:L_0805_2012Metric -> PCM_Ferrite_SMD_AKL:Ferrite_0805_2012Metric
- FB402: renamed from FB702; footprint Inductor_SMD:L_0805_2012Metric -> PCM_Ferrite_SMD_AKL:Ferrite_0805_2012Metric
- FB403: renamed from FB703; footprint Inductor_SMD:L_0805_2012Metric -> PCM_Ferrite_SMD_AKL:Ferrite_0805_2012Metric
- FB501: renamed from FB801; footprint Inductor_SMD:L_0805_2012Metric -> PCM_Ferrite_SMD_AKL:Ferrite_0805_2012Metric
- FB801: renamed from FB401; footprint Inductor_SMD:L_0805_2012Metric -> PCM_Ferrite_SMD_AKL:Ferrite_0805_2012Metric
- G601: footprint HALMET:cc-by_5mm -> HALSER:cc-by_5mm
- G605: footprint HALMET:Hat_Labs_25.4mm -> HALSER:Hat_Labs_25.4mm
- G606: renamed from G701; footprint HALMET:HaL_picto_8mm -> HALSER:HaL_picto_8mm
- H601: renamed from H1001; footprint HALMET:MountingSlot_3.2mm_M3_Unplated -> MountingHole:MountingHole_3.2mm_M3_ISO7380
- H602: renamed from H1002; footprint HALMET:MountingSlot_3.2mm_M3_Unplated -> MountingHole:MountingHole_3.2mm_M3_ISO7380
- J401: renamed from J702; value Conn_01x04 -> I2C Female Header
- J501: renamed from J801; value Conn_01x03 -> 1-Wire Male Header
- J802: value Conn_01x04 -> USB_C_Receptacle_USB2.0_16P; footprint Connector_Phoenix_MC:PhoenixContact_MCV_1,5_4-G-3.81_1x04_P3.81mm_Vertical -> HALSER:Shou Han Type-C 16P LTH6.8
- J901: renamed from J1201; value Conn_01x02 -> 3V3 Header
- L701: value NLCV32T-100K-EFR -> CBC3225T100KR
- L702: renamed from L301; value SMMS0650-470M -> SLO0530H6R8MTT; footprint HALMET:SMMS0650-1R0M -> Inductor_SMD:L_Chilisin_BMRA00050530
- R1001, R1002: footprint Resistor_SMD:R_0402_1005Metric -> PCM_Resistor_SMD_AKL:R_0402_1005Metric
- R203: renamed from R503; footprint Resistor_SMD:R_0402_1005Metric -> PCM_Resistor_SMD_AKL:R_0402_1005Metric
- R204: renamed from R213; footprint Resistor_SMD:R_0402_1005Metric -> PCM_Resistor_SMD_AKL:R_0402_1005Metric
- R301: renamed from R1103; footprint Resistor_SMD:R_0402_1005Metric -> PCM_Resistor_SMD_AKL:R_0402_1005Metric
- R302: renamed from R201; footprint Resistor_SMD:R_0402_1005Metric -> PCM_Resistor_SMD_AKL:R_0402_1005Metric
- R401: renamed from R701; footprint Resistor_SMD:R_0402_1005Metric -> PCM_Resistor_SMD_AKL:R_0402_1005Metric
- R402: renamed from R702; footprint Resistor_SMD:R_0402_1005Metric -> PCM_Resistor_SMD_AKL:R_0402_1005Metric
- R501: renamed from R801; footprint Resistor_SMD:R_0402_1005Metric -> PCM_Resistor_SMD_AKL:R_0402_1005Metric
- R502: renamed from R802; footprint Resistor_SMD:R_0805_2012Metric -> PCM_Resistor_SMD_AKL:R_0805_2012Metric
- R703: value 4.7R -> 24k; footprint Resistor_SMD:R_0603_1608Metric -> PCM_Resistor_SMD_AKL:R_0402_1005Metric
- R901: renamed from R1201; footprint Resistor_SMD:R_0402_1005Metric -> PCM_Resistor_SMD_AKL:R_0402_1005Metric
- U201: renamed from U501; footprint Package_SO:SOIC-8_3.9x4.9mm_P1.27mm -> PCM_Package_SO_AKL:SOIC-8_3.9x4.9mm_P1.27mm
- U902: renamed from U1203; footprint Package_TO_SOT_SMD:SOT-23-3 -> PCM_Package_TO_SOT_SMD_AKL:SOT-23
- moved G601 118.2 mm to (273.0, 158.0)
- moved G602 118.2 mm to (263.9, 122.8)
- moved G605 118.2 mm to (239.4, 149.2)
- moved G606 115.3 mm to (243.2, 158.0)
- moved J802 64.5 mm to (166.6, 87.5), turned to 90 degrees
- moved D701 49.2 mm to (160.7, 101.1), turned to 90 degrees
- moved F701 48.5 mm to (147.7, 107.0)
- moved D1002 47.7 mm to (120.4, 59.4), turned to -90 degrees
- moved D501 47.7 mm to (160.2, 65.5)
- moved C502 47.2 mm to (161.5, 61.6), turned to 180 degrees
- moved R502 47.0 mm to (161.5, 63.6), turned to 180 degrees
- moved D1001 46.3 mm to (118.2, 59.4), turned to 90 degrees
- moved D702 45.9 mm to (147.1, 111.6)
- moved D502 45.5 mm to (153.1, 65.6)
- moved J501 45.4 mm to (154.4, 68.0), turned to 90 degrees
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- renumbered L1201 to L901, L1202 to L902, PS1201 to PS901
Connections:
- net /ESP32/EN renamed /ESP32/CHIP_PU
- C707 pad 1: /Power input/IN -> /Power input/SW
- C707 pad 2: GND -> /Power input/CB
- C708 pad 1: /Power input/IN -> +3.3V
- C709 pad 1: /Power input/IN -> +3.3V
- D1001 pad 1: /CAN_RX -> /Isolation barrier/iVIA
- D1002 pad 1: /CAN_TX -> /Isolation barrier/iVOB
- D802 pad 2: /USB/USB_D+ -> /USB_D-
- D803 pad 2: /USB/USB_D- -> /USB_D+
- F701 pad 2: /Power input/CAN_+ -> /Power input/Vin
- L701 pad 2: Net-(C713-Pad1) -> /Power input/IN
- R1001 pad 1: +3.3V -> +3.3V_1
- R1002 pad 1: +3.3V -> +3.3V_1
- R301 pad 2: /ESP32/IO0 -> /ESP32/GPIO8
- R703 pad 1: GND -> /Power input/FB
- R703 pad 2: Net-(C716-Pad2) -> GND
- U201 pad 6: /CAN_L -> Net-(D201-A1)
- U201 pad 7: /CAN_H -> Net-(D201-A2)
Routing:
- net +3.3V_1: track 250.0 -> 0.00 mm, vias 23 -> 0
- net GND: track 123.0 -> 2.03 mm, vias 65 -> 0
- net USB_5V: track 82.9 -> 0.00 mm, vias 5 -> 0
- net /SCL: track 68.4 -> 0.00 mm, vias 6 -> 0
- net +3.3V: track 241.9 -> 176.0 mm, vias 22 -> 15
- net GND1: track 63.6 -> 0.00 mm, vias 41 -> 0
- net /Digital input/DigIn1: track 58.4 -> 0.00 mm, vias 4 -> 0
- net /SDA: track 57.7 -> 0.00 mm, vias 5 -> 0
- net Net-(U601C--): track 51.0 -> 0.00 mm, vias 4 -> 0
- net /Analog input/ADC_A1: track 48.1 -> 0.00 mm, vias 2 -> 0
- net Net-(U601A--): track 47.7 -> 0.00 mm, vias 4 -> 0
- net /Digital input/DigIn2: track 47.4 -> 0.00 mm, vias 4 -> 0
- net /LED: track 42.3 -> 0.00 mm, vias 2 -> 0
- net /DI1: track 41.7 -> 0.00 mm, vias 4 -> 0
- net /ESP32/CHIP_PU: track 40.9 -> 0.00 mm, vias 3 -> 0
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- removed copper zone on In1.Cu, net GND1
- removed copper zone on In2.Cu, net GND1
Other:
- board size 89 x 58 mm -> 90.8 x 58.8 mm
- board text added: "0.96{dblquote} Display Outline"
- board text added: "A"
- board text added: "B"
- board text added: "Edge margin 10 mm; no connectors!"
- board text added: "R"
- board text added: "T"
- board text removed: "ANTENNA-KEEP OUT"
- board text removed: "USB impedance controlled traces designed for the JLC7628 stackup"

Commit message: Further design adjustments
Parts:
- removed J901: 3V3 Header, Connector_PinHeader_2.54mm:PinHeader_1x02_P2.54mm_Vertical
- removed the REF** at (134.0, 56.6)
- removed the REF** at (179.4, 97.3)
- removed the REF** at (134.0, 115.4)
- removed the REF** at (88.6, 86.0)
- added J402: I2C Male Header, Connector_PinHeader_2.54mm:PinHeader_1x04_P2.54mm_Vertical, F.Cu at (133.0, 79.4)
- added J702: Vin header, Connector_PinHeader_2.54mm:PinHeader_1x02_P2.54mm_Vertical, F.Cu at (155.9, 122.5)
- added J703: CAN Header, Connector_PinHeader_2.54mm:PinHeader_1x04_P2.54mm_Vertical, F.Cu at (148.2, 114.9)
- added REF**: ProtoPad_1x01_P2.54_2.0x2.0, HALSER:ProtoPad_1x01_P2.54_2.0x2.0, F.Cu at (105.1, 130.2)
- added REF**: ProtoPad_1x04_P2.54_2.1x2.1_Octagonal, HALSER:ProtoPad_1x04_P2.54_2.1x2.1_Octagonal, F.Cu at (145.7, 79.4)
- added REF**: ProtoPad_1x01_P2.54_2.0x2.0, HALSER:ProtoPad_1x01_P2.54_2.0x2.0, F.Cu at (176.2, 112.4)
- added REF**: ProtoPad_1x02_P2.54_2.1x2.1_Octagonal, HALSER:ProtoPad_1x02_P2.54_2.1x2.1_Octagonal, F.Cu at (176.2, 114.9)
- added REF**: ProtoPad_1x01_P2.54_D2.0, HALSER:ProtoPad_1x01_P2.54_D2.0, F.Cu at (173.6, 112.4)
- added REF**: ProtoPad_1x01_P2.54_2.0x2.0, HALSER:ProtoPad_1x01_P2.54_2.0x2.0, F.Cu at (160.9, 132.7)
- added REF**: ProtoPad_1x01_P2.54_D2.0, HALSER:ProtoPad_1x01_P2.54_D2.0, F.Cu at (105.1, 132.7)
- added REF**: ProtoPad_1x01_P2.54_D2.0, HALSER:ProtoPad_1x01_P2.54_D2.0, F.Cu at (160.9, 130.2)
- added REF**: ProtoPad_1x02_P2.54_2.1x2.1_Octagonal, HALSER:ProtoPad_1x02_P2.54_2.1x2.1_Octagonal, F.Cu at (102.5, 132.7)
- added REF**: Tab, PCM_kikit:Tab, F.Cu at (179.5, 106.0)
- added REF**: ProtoPad_1x02_P2.54_2.1x2.1_Octagonal, HALSER:ProtoPad_1x02_P2.54_2.1x2.1_Octagonal, F.Cu at (168.6, 132.7)
- added REF**: ProtoPad_1x02_P2.54_2.1x2.1_Octagonal, HALSER:ProtoPad_1x02_P2.54_2.1x2.1_Octagonal, F.Cu at (163.5, 132.7)
- added REF**: Tab, PCM_kikit:Tab, F.Cu at (134.0, 135.5)
- added REF**: ProtoPad_1x04_P2.54_2.1x2.1_Octagonal, HALSER:ProtoPad_1x04_P2.54_2.1x2.1_Octagonal, F.Cu at (160.9, 79.4)
- added REF**: Tab, PCM_kikit:Tab, F.Cu at (88.5, 106.0)
- added REF**: ProtoPad_1x02_P2.54_2.1x2.1_Octagonal, HALSER:ProtoPad_1x02_P2.54_2.1x2.1_Octagonal, F.Cu at (176.2, 122.5)
- added REF**: ProtoPad_1x02_P2.54_2.1x2.1_Octagonal, HALSER:ProtoPad_1x02_P2.54_2.1x2.1_Octagonal, F.Cu at (158.4, 79.4)
- added REF**: ProtoPad_1x02_P2.54_2.1x2.1_Octagonal, HALSER:ProtoPad_1x02_P2.54_2.1x2.1_Octagonal, F.Cu at (100.0, 132.7)
- added REF**: Tab, PCM_kikit:Tab, F.Cu at (134.0, 76.5)
- added REF**: ProtoPad_1x02_P2.54_2.1x2.1_Octagonal, HALSER:ProtoPad_1x02_P2.54_2.1x2.1_Octagonal, F.Cu at (176.2, 117.5)
- added REF**: ProtoPad_1x02_P2.54_2.1x2.1_Octagonal, HALSER:ProtoPad_1x02_P2.54_2.1x2.1_Octagonal, F.Cu at (176.2, 120.0)
- added REF**: ProtoPad_1x02_P2.54_2.1x2.1_Octagonal, HALSER:ProtoPad_1x02_P2.54_2.1x2.1_Octagonal, F.Cu at (166.0, 132.7)
- added REF**: ProtoPad_1x02_P2.54_2.1x2.1_Octagonal, HALSER:ProtoPad_1x02_P2.54_2.1x2.1_Octagonal, F.Cu at (176.2, 125.1)
- G603: moved to B.Cu
- R306: footprint PCM_Resistor_SMD_AKL:R_0603_1608Metric -> PCM_Resistor_SMD_AKL:R_0603_1608Metric_Pad0.98x0.95mm_HandSolder
- moved G602 144.5 mm to (119.5, 126.6)
- moved G603 144.0 mm to (132.1, 127.0), turned to 180 degrees
- moved G606 127.5 mm to (118.7, 130.8)
- moved G605 116.8 mm to (134.9, 97.2)
- moved G601 113.1 mm to (164.9, 124.6)
- moved D302 31.4 mm to (140.0, 108.4)
- moved D303 31.4 mm to (148.5, 108.4)
- moved R901 28.9 mm to (113.7, 87.6), turned to 90 degrees
- moved C1015 26.9 mm to (107.8, 119.9), turned to 0 degrees
- moved D1009 26.9 mm to (107.3, 118.3), turned to 180 degrees
- moved FB1002 25.9 mm to (107.7, 121.9), turned to 180 degrees
- moved R801 25.6 mm to (161.1, 110.3), turned to -90 degrees
- moved C1013 25.0 mm to (107.4, 123.9)
- moved D802 25.0 mm to (162.3, 110.3), turned to 90 degrees
- moved D803 24.4 mm to (168.6, 110.3), turned to 90 degrees
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Connections:
- net /Power input/IN renamed /Power input/VIN
- net /Serial interfaces/RS232_RX_LINE renamed /Serial interfaces/RS232_RX_C
- net /Serial interfaces/RS232_TX_LINE renamed /Serial interfaces/RS232_TX_C
- net /Serial interfaces/RS485_RX_A_LINE renamed /Serial interfaces/RS485_RX_B_C
- net /Serial interfaces/RS485_RX_B_LINE renamed /Serial interfaces/RS485_RX_A_C
- net /Serial interfaces/RS485_TX_A_LINE renamed /Serial interfaces/RS485_TX_A_C
- net /Serial interfaces/RS485_TX_B_LINE renamed /Serial interfaces/RS485_TX_B_C
- net Net-(D1007-A2) renamed /Serial interfaces/UART_TX_C
- net Net-(D1009-A2) renamed /Serial interfaces/UART_RX_C
- net Net-(J802-CC1) renamed /USB/CC1
- net Net-(J802-CC2) renamed /USB/CC2
- C402 pad 1: /I2C/SDA_CONN -> /SDA_C
- C403 pad 1: /I2C/SCL_CONN -> /SCL_C
- D302 pad 1: /CAN_RX -> Net-(D302-K)
- D302 pad 2: Net-(D302-A) -> +3.3V
- D401 pad 2: /I2C/SDA_CONN -> /SDA_C
- D402 pad 2: /I2C/SCL_CONN -> /SCL_C
- D501 pad 2: /Onewire/DQ_CONN -> /DQ_C
- FB402 pad 1: /I2C/SDA_CONN -> /SDA_C
- FB403 pad 1: /I2C/SCL_CONN -> /SCL_C
- J301 pad 15: /DQ -> /DQ_C
- J301 pad 17: /SDA -> /ESP32/GPIO0
- J301 pad 19: /SCL -> /ESP32/GPIO1
- J301 pad 5: /ESP32/GPIO0 -> /SDA_C
- J301 pad 7: /ESP32/GPIO1 -> /SCL_C
- J401 pad 3: /I2C/SCL_CONN -> /SCL_C
- J401 pad 4: /I2C/SDA_CONN -> /SDA_C
- J501 pad 3: /Onewire/DQ_CONN -> /DQ_C
- R304 pad 1: +3.3V -> Net-(D302-K)
- R304 pad 2: Net-(D302-A) -> /CAN_RX
- R502 pad 2: /Onewire/DQ_CONN -> /DQ_C
Routing:
- net +3.3V_1: track 0.00 -> 127.4 mm, vias 0 -> 14
- net GND: track 2.03 -> 129.2 mm, vias 0 -> 132
- net /Isolation barrier/iVOB: track 0.00 -> 75.0 mm, vias 0 -> 8
- net +3.3V: track 176.0 -> 235.5 mm, vias 15 -> 25
- net /ESP32/CHIP_PU: track 0.00 -> 55.4 mm, vias 0 -> 4
- net /Isolation barrier/iVIA: track 0.00 -> 53.7 mm, vias 0 -> 3
- net /SCL_C: track 0.00 -> 50.8 mm, vias 0 -> 2
- net /ESP32/GPIO9: track 0.00 -> 46.7 mm, vias 0 -> 6
- net /Serial interfaces/UART_RX: track 0.00 -> 41.5 mm, vias 0 -> 2
- net /SCL: track 0.00 -> 40.9 mm, vias 0 -> 4
- net /SDA_C: track 0.00 -> 40.0 mm, vias 0 -> 1
- net /DQ_C: track 0.00 -> 39.2 mm, vias 0 -> 1
- net GND1: track 0.00 -> 38.3 mm, vias 0 -> 69
- net /SDA: track 0.00 -> 36.5 mm, vias 0 -> 4
- net /ESP32/GPIO1: track 0.00 -> 34.1 mm, vias 0 -> 4
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- added copper zone on In1.Cu, net GND1
- added copper zone on In2.Cu, net GND1
Other:
- outline, holes or cut-outs redrawn
- board text added: "0"
- board text added: "1"
- board text added: "12V"
- board text added: "20"
- board text added: "21"
- board text added: "6"
- board text added: "9"
- board text added: "BTN"
- board text added: "CRX"
- board text added: "CTX"
- board text added: "HALSER"
- board text added: "L H 12V GND"
- board text added: "LE"
- board text added: "N"
- board text added: "N183 RX"
- board text added: "N183 TX"
- board text added: "RES"
- board text added: "RGB"
- board text added: "RS-232"
- board text added: "RX SEL"
- board text added: "SRX"
- board text added: "STX"
- board text added: "Serial Interface Board"
- board text added: "U"
- board text added: "UART"
- board text added: "VIN"
- board text added: "i3V3"
- board text added: "iGND"
- board text added: "v1.0.0-a1"
- board text removed: "+"
- board text removed: "-"
- board text removed: "00 BOOT"
- board text removed: "01 TXD0"
- board text removed: "02 LED"
- board text removed: "03 RXD0"
- board text removed: "04 1-WIRE"
- board text removed: "0x48"
- board text removed: "0x49"
- board text removed: "0x4a"
- board text removed: "0x4b"
- board text removed: "12"
- board text removed: "12 TDI"
- board text removed: "13"
- board text removed: "13 TCK"
- board text removed: "14"
- board text removed: "14 TMS"
- board text removed: "15"
- board text removed: "15 TDO"
- board text removed: "16"
- board text removed: "17"
- board text removed: "18 CAN_RX"
- board text removed: "19 CAN_TX"
- board text removed: "21 SDA"
- board text removed: "22 SCL"
- board text removed: "23 DI1"
- board text removed: "25 DI2"
- board text removed: "26 DI4"
- board text removed: "27 DI3"
- board text removed: "32"
- board text removed: "33"
- board text removed: "34"
- board text removed: "35"
- board text removed: "5"
- board text removed: "A1"
- board text removed: "A2"
- board text removed: "A3"
- board text removed: "A4"
- board text removed: "ADS1115 address"
- board text removed: "Analog"
- board text removed: "BOOT"
- board text removed: "Black"
- board text removed: "Blue"
- board text removed: "CAN term."
- board text removed: "CCS"
- board text removed: "D1"
- board text removed: "D2"
- board text removed: "D3"
- board text removed: "D4"
- board text removed: "Digital"
- board text removed: "EN"
- board text removed: "GPIO"
- board text removed: "GPIO FUNC"
- board text removed: "GPIO JTAG"
- board text removed: "HALMET"
- board text removed: "IN"
- board text removed: "IO0"
- board text removed: "Input 6-32V"
- board text removed: "LP"
- board text removed: "Marine Engine & Tank Interface"
- board text removed: "PDN"
- board text removed: "PUP"
- board text removed: "RESET"
- board text removed: "Red"
- board text removed: "T"
- board text removed: "USB"
- board text removed: "USB 5V"
- board text removed: "VN"
- board text removed: "VP"
- board text removed: "White"
- board text removed: "v1.0.1"

Commit message: Further manufacturing tweaks
Parts:
- C904: value 220pF/2kV -> 1nF/X1,Y2
Routing:
- net /ESP32/GPIO9: track 46.7 -> 47.8 mm
- net /SCL: track 40.9 -> 40.4 mm

Commit message: FIXUP vias
Routing:
- net /SER_RX: track 55.4 -> 56.0 mm
- net GND: vias 132 -> 130
Changed lines of the file:
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@@
 	)
 	(via
-		(at 166.625 104.1)
-		(size 0.45)
-		(drill 0.2)
-		(layers "F.Cu" "B.Cu")
-		(free yes)
-		(net 1)
-	)
-	(via
 		(at 160.625 100.7)
 		(size 0.45)
@@
 	)
 	(via
-		(at 164.325 104)
-		(size 0.45)
-		(drill 0.2)
-		(layers "F.Cu" "B.Cu")
-		(free yes)
-		(net 1)
-	)
-	(via
 		(at 127.782 128.205441)
 		(size 0.8)
@@
 	)
 	(segment
-		(start 165.75 105.1)
-		(end 165.75 104.15)
+		(start 164.775 100.3)
+		(end 164.775 102.826471)
+		(width 0.25)
+		(layer "F.Cu")
+		(net 38)
+	)
+	(segment
+		(start 165.75 104.05)
+		(end 165.775 104.025)
 		(width 0.25)
 		(layer "F.Cu")
@@
 	)
 	(segment
-		(start 164.775 103.175)
-		(end 164.775 100.3)
+		(start 164.775 102.826471)
+		(end 165.775 103.826471)
 		(width 0.25)
 		(layer "F.Cu")
@@
 	)
 	(segment
-		(start 165.25 106.317061)
-		(end 165.250003 106.317058)
+		(start 165.75 105.1)
+		(end 165.75 104.05)
 		(width 0.25)
 		(layer "F.Cu")
@@
 	)
 	(segment
-		(start 165.25 106.865)
-		(end 165.25 107.704595)
+		(start 165.775 103.826471)
+		(end 165.775 104.025)
 		(width 0.25)
 		(layer "F.Cu")
@@
 	)
 	(segment
-		(start 165.75 104.15)
-		(end 164.775 103.175)
+		(start 165.25 106.317061)
+		(end 165.250003 106.317058)
+		(width 0.25)
+		(layer "F.Cu")
+		(net 38)
+	)
+	(segment
+		(start 165.25 106.865)
+		(end 165.25 107.704595)
 		(width 0.25)
 		(layer "F.Cu")
@@
 	)
 	(via
-		(at 165.75 104.15)
+		(at 165.775 104.025)
 		(size 0.45)
 		(drill 0.2)
@@
 	)
 	(segment
-		(start 165.75 104.15)
-		(end 165.75 105.817061)
+		(start 165.775 105.792061)
+		(end 165.775 104.025)
 		(width 0.25)
 		(layer "B.Cu")
@@
 	)
 	(segment
-		(start 165.75 105.817061)
-		(end 165.250003 106.317058)
+		(start 165.250003 106.317058)
+		(end 165.775 105.792061)
 		(width 0.25)
 		(layer "B.Cu")
@@
 	)
 	(segment
-		(start 165.575 100.3)
-		(end 165.575 102.875)
+		(start 165.25 105.1)
+		(end 165.25 104.25)
 		(width 0.25)
 		(layer "F.Cu")
@@
 	)
 	(segment
-		(start 165.575 102.875)
-		(end 165.6 102.9)
+		(start 165.575 102.67647)
+		(end 165.699265 102.800735)
 		(width 0.25)
 		(layer "F.Cu")
@@
 	)
 	(segment
-		(start 165.25 104.375337)
-		(end 165.074663 104.2)
+		(start 165.575 100.3)
+		(end 165.575 102.67647)
 		(width 0.25)
 		(layer "F.Cu")
@@
 	)
 	(segment
-		(start 165.25 105.1)
-		(end 165.25 104.375337)
+		(start 165.848 106.767)
+		(end 165.848 106.178)
 		(width 0.25)
 		(layer "F.Cu")
@@
 	)
 	(segment
-		(start 165.848 106.767)
-		(end 165.848 106.178)
+		(start 165.25 104.25)
+		(end 165.075 104.075)
 		(width 0.25)
 		(layer "F.Cu")
@@
 	)
 	(via
-		(at 165.6 102.9)
+		(at 165.699265 102.800735)
 		(size 0.45)
 		(drill 0.2)
@@
 	)
 	(via
-		(at 165.074663 104.2)
+		(at 165.075 104.075)
 		(size 0.45)
 		(drill 0.2)
@@
 	)
 	(segment
-		(start 165.074663 104.2)
-		(end 165.074663 103.425337)
+		(start 165.699265 102.800735)
+		(end 165.075 103.425)
 		(width 0.25)
 		(layer "B.Cu")
@@
 	)
 	(segment
-		(start 165.074663 103.425337)
-		(end 165.6 102.9)
+		(start 165.075 103.425)
+		(end 165.075 104.075)
 		(width 0.25)
 		(layer "B.Cu")
@@
 	)
 	(segment
+		(start 168.775 88.85)
+		(end 169.225 89.3)
+		(width 0.25)
+		(layer "F.Cu")
+		(net 56)
+	)
+	(segment
 		(start 159.95 96.763173)
 		(end 159.95 99.65)
@@
 	)
 	(segment
-		(start 168.775 88.5)
-		(end 168.775 89.25)
-		(width 0.25)
+		(start 159.95 99.65)
+		(end 157.025002 102.574998)
+		(width 0.2)
 		(layer "F.Cu")
 		(net 56)
 	)
 	(segment
-		(start 159.95 99.65)
-		(end 157.025002 102.574998)
-		(width 0.2)
+		(start 168.775 88.5)
+		(end 168.775 88.85)
+		(width 0.25)
 		(layer "F.Cu")
 		(net 56)
@@
 	)
 	(via
-		(at 168.775 89.25)
+		(at 169.225 89.3)
 		(size 0.45)
 		(drill 0.2)
@@
 	)
 	(segment
-		(start 156.311109 103.297)
-		(end 157.025002 102.583107)
-		(width 0.2)
-		(layer "B.Cu")
-		(net 56)
-	)
-	(segment
-		(start 154.788 103.297)
-		(end 156.311109 103.297)
-		(width 0.2)
+		(start 164.802 93.498)
+		(end 169 89.3)
+		(width 0.25)
 		(layer "B.Cu")
 		(net 56)
 	)
 	(segment
-		(start 133.35 94.3)
-		(end 133.95 93.7)
+		(start 134.152 93.498)
+		(end 164.802 93.498)
 		(width 0.25)
 		(layer "B.Cu")
@@
 	)
 	(segment
-		(start 157.025002 102.583107)
-		(end 157.025002 102.574998)
+		(start 156.311109 103.297)
+		(end 157.025002 102.583107)
 		(width 0.2)
 		(layer "B.Cu")
@@
 	)
 	(segment
-		(start 152.223 93.498)
-		(end 164.527 93.498)
+		(start 169 89.3)
+		(end 169.225 89.3)
 		(width 0.25)
 		(layer "B.Cu")
@@
 	)
 	(segment
-		(start 133.95 93.7)
-		(end 152.021 93.7)
-		(width 0.25)
+		(start 154.788 103.297)
+		(end 156.311109 103.297)
+		(width 0.2)
 		(layer "B.Cu")
 		(net 56)
 	)
 	(segment
-		(start 152.021 93.7)
-		(end 152.223 93.498)
-		(width 0.25)
+		(start 157.025002 102.583107)
+		(end 157.025002 102.574998)
+		(width 0.2)
 		(layer "B.Cu")
 		(net 56)
 	)
 	(segment
-		(start 164.527 93.498)
-		(end 168.775 89.25)
+		(start 133.35 94.3)
+		(end 134.152 93.498)
 		(width 0.25)
 		(layer "B.Cu")
@@
 		(polygon
 			(pts
-				(xy 173.575 82.05) (xy 180.125 82.05) (xy 180.125 101.8) (xy 173.575 101.8)
+				(xy 173.575 82.05) (xy 180.125 82.05) (xy 180.125 102.725) (xy 173.575 102.725)
 			)
 		)
