File: HALSER.kicad_sch (KiCad schematic)
At the start: 0 parts

Commit message: Redo schematics
Other:
- removed sheet Analog input
- removed sheet Digital input
- removed sheet User Interface
- added sheet Serial interfaces (serial.kicad_sch)
- sheet ESP32 ports: added SER_RX, SER_TX, USB_D+, USB_D-; removed BOOT_AUTO, BOOT_KEY, DI1, DI2, DI3, DI4, IO2, RESET_AUTO, RESET_KEY, USB_RXD, USB_TXD
- sheet Isolation barrier ports: added VIB, iVOB; removed SCL1, SDA1, VOB, VOC, VOD, iSCL, iSDA, iVIB, iVIC, iVID
- sheet USB ports: added USB_D+, USB_D-; removed BOOT_AUTO, RESET_AUTO, RXD, TXD

Commit message: Further design adjustments
Other:
- sheet ESP32 ports: added DQ_C, SCL_C, SDA_C; removed none
- sheet I2C ports: added SCL_C, SDA_C; removed none
- sheet Onewire ports: added DQ_C; removed none

Commit message: Fix issues found in -a1
Other:
- company: Hat Labs Ltd -> Hat Labs oy
- title: Hat Labs Marine Engine & Tank interface (HALMET) -> Hat Labs Serial Interface Device (HALSER)
Changed lines of the file:
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@@
 	(paper "A4")
 	(title_block
-		(title "Hat Labs Marine Engine & Tank interface (HALMET)")
-		(date "2024-01-18")
-		(rev "1.0.1")
-		(company "Hat Labs Ltd")
+		(title "Hat Labs Serial Interface Device (HALSER)")
+		(date "2024-11-20")
+		(rev "1.0.0-a1")
+		(company "Hat Labs oy")
 		(comment 1 "https://creativecommons.org/licenses/by-sa/4.0")
 		(comment 2 "To view a copy of this license, visit ")
