File: I2C.kicad_sch (KiCad schematic)
At the start: 15 parts, among them J702 Conn_01x04

Commit message: Redo schematics
Parts:
- C401: renamed from C704; footprint Capacitor_SMD:C_1206_3216Metric -> PCM_Capacitor_SMD_AKL:C_1206_3216Metric
- C402: renamed from C705; footprint Capacitor_SMD:C_0603_1608Metric -> PCM_Capacitor_SMD_AKL:C_0603_1608Metric
- C403: renamed from C706; footprint Capacitor_SMD:C_0603_1608Metric -> PCM_Capacitor_SMD_AKL:C_0603_1608Metric
- C404: renamed from C701; footprint Capacitor_SMD:C_0402_1005Metric -> PCM_Capacitor_SMD_AKL:C_0603_1608Metric; LCSC C15525 -> C19702
- C405: renamed from C702; footprint Capacitor_SMD:C_0402_1005Metric -> PCM_Capacitor_SMD_AKL:C_0402_1005Metric
- C406: renamed from C703; footprint Capacitor_SMD:C_0402_1005Metric -> PCM_Capacitor_SMD_AKL:C_0402_1005Metric
- D401, D402, D403: footprint Diode_SMD:D_0402_1005Metric -> PCM_Diode_SMD_AKL:D_0402_1005Metric
- FB401: renamed from FB701; footprint Inductor_SMD:L_0805_2012Metric -> PCM_Ferrite_SMD_AKL:Ferrite_0805_2012Metric
- FB402: renamed from FB702; footprint Inductor_SMD:L_0805_2012Metric -> PCM_Ferrite_SMD_AKL:Ferrite_0805_2012Metric
- FB403: renamed from FB703; footprint Inductor_SMD:L_0805_2012Metric -> PCM_Ferrite_SMD_AKL:Ferrite_0805_2012Metric
- J401: renamed from J702; value Conn_01x04 -> I2C Female Header
- R401: renamed from R701; footprint Resistor_SMD:R_0402_1005Metric -> PCM_Resistor_SMD_AKL:R_0402_1005Metric
- R402: renamed from R702; footprint Resistor_SMD:R_0402_1005Metric -> PCM_Resistor_SMD_AKL:R_0402_1005Metric

Commit message: Further design adjustments
Parts:
- added J402: I2C Male Header, Connector_PinHeader_2.54mm:PinHeader_1x04_P2.54mm_Vertical, symbol Connector_Generic:Conn_01x04
Connections:
- net GND: now also J402.1 (Pin_1)
- net I2C_3V3: now also J402.2 (Pin_2)
- net SCL_CONN renamed SCL_C
- net SCL_C: now also J402.3 (Pin_3)
- net SDA_CONN renamed SDA_C
- net SDA_C: now also J402.4 (Pin_4)

Commit message: Further manufacturing tweaks
Parts:
- J401: LCSC C124413 -> C2718488
- J402: LCSC C7430360 -> C6332197
Changed lines of the file:
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@@
 			)
 		)
-		(property "LCSC" "C124413"
+		(property "LCSC" "C2718488"
 			(at 41.91 85.09 0)
 			(effects
@@
 			)
 		)
-		(property "LCSC" "C7430360"
+		(property "LCSC" "C6332197"
 			(at 41.91 69.85 0)
 			(effects

Commit message: Fix issues found in -a1
Parts:
- C401: footprint PCM_Capacitor_SMD_AKL:C_1206_3216Metric -> Capacitor_SMD:C_1206_3216Metric
- C402, C403, C404: footprint PCM_Capacitor_SMD_AKL:C_0603_1608Metric -> Capacitor_SMD:C_0603_1608Metric
- C405, C406: footprint PCM_Capacitor_SMD_AKL:C_0402_1005Metric -> Capacitor_SMD:C_0402_1005Metric
- D401, D402, D403: footprint PCM_Diode_SMD_AKL:D_0402_1005Metric -> Diode_SMD:D_0402_1005Metric
- FB401, FB402, FB403: footprint PCM_Ferrite_SMD_AKL:Ferrite_0805_2012Metric -> Inductor_SMD:L_0805_2012Metric
- R401, R402: footprint PCM_Resistor_SMD_AKL:R_0402_1005Metric -> Resistor_SMD:R_0402_1005Metric
Other:
- company: Hat Labs Ltd -> Hat Labs oy
- title: Hat Labs Marine Engine & Tank interface (HALMET) -> Hat Labs Serial Interface Device (HALSER)
Changed lines of the file:
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@@
 	(paper "A4")
 	(title_block
-		(title "Hat Labs Marine Engine & Tank interface (HALMET)")
-		(date "2024-01-18")
-		(rev "1.0.1")
-		(company "Hat Labs Ltd")
+		(title "Hat Labs Serial Interface Device (HALSER)")
+		(date "2024-11-20")
+		(rev "1.0.0-a1")
+		(company "Hat Labs oy")
 		(comment 1 "https://creativecommons.org/licenses/by-sa/4.0")
 		(comment 2 "To view a copy of this license, visit ")
@@
 			)
 		)
-		(property "Footprint" "PCM_Capacitor_SMD_AKL:C_0603_1608Metric"
+		(property "Footprint" "Capacitor_SMD:C_0603_1608Metric"
 			(at 136.1948 116.84 0)
 			(effects
@@
 			)
 		)
-		(property "Footprint" "PCM_Capacitor_SMD_AKL:C_0603_1608Metric"
+		(property "Footprint" "Capacitor_SMD:C_0603_1608Metric"
 			(at 136.1948 96.52 0)
 			(effects
@@
 			)
 		)
-		(property "Footprint" "PCM_Capacitor_SMD_AKL:C_0402_1005Metric"
+		(property "Footprint" "Capacitor_SMD:C_0402_1005Metric"
 			(at 149.5552 96.52 0)
 			(effects
@@
 			)
 		)
-		(property "Footprint" "PCM_Capacitor_SMD_AKL:C_0402_1005Metric"
+		(property "Footprint" "Capacitor_SMD:C_0402_1005Metric"
 			(at 149.5552 116.84 0)
 			(effects
@@
 			)
 		)
-		(property "Footprint" "PCM_Capacitor_SMD_AKL:C_1206_3216Metric"
+		(property "Footprint" "Capacitor_SMD:C_1206_3216Metric"
 			(at 136.1948 76.2 0)
 			(effects
@@
 			)
 		)
-		(property "Footprint" "PCM_Capacitor_SMD_AKL:C_0603_1608Metric"
+		(property "Footprint" "Capacitor_SMD:C_0603_1608Metric"
 			(at 149.5552 76.2 0)
 			(effects
@@
 			)
 		)
-		(property "Footprint" "PCM_Resistor_SMD_AKL:R_0402_1005Metric"
+		(property "Footprint" "Resistor_SMD:R_0402_1005Metric"
 			(at 83.82 49.022 90)
 			(effects
@@
 			)
 		)
-		(property "Footprint" "PCM_Resistor_SMD_AKL:R_0402_1005Metric"
+		(property "Footprint" "Resistor_SMD:R_0402_1005Metric"
 			(at 83.82 55.372 90)
 			(effects
@@
 			)
 		)
-		(property "Footprint" "PCM_Ferrite_SMD_AKL:Ferrite_0805_2012Metric"
+		(property "Footprint" "Inductor_SMD:L_0805_2012Metric"
 			(at 142.24 66.802 90)
 			(effects
@@
 			)
 		)
-		(property "Footprint" "PCM_Ferrite_SMD_AKL:Ferrite_0805_2012Metric"
+		(property "Footprint" "Inductor_SMD:L_0805_2012Metric"
 			(at 142.24 107.442 90)
 			(effects
@@
 			)
 		)
-		(property "Footprint" "PCM_Ferrite_SMD_AKL:Ferrite_0805_2012Metric"
+		(property "Footprint" "Inductor_SMD:L_0805_2012Metric"
 			(at 142.24 87.122 90)
 			(effects
@@
 			)
 		)
-		(property "Footprint" "PCM_Diode_SMD_AKL:D_0402_1005Metric"
+		(property "Footprint" "Diode_SMD:D_0402_1005Metric"
 			(at 85.09 97.79 0)
 			(effects
@@
 			)
 		)
-		(property "Footprint" "PCM_Diode_SMD_AKL:D_0402_1005Metric"
+		(property "Footprint" "Diode_SMD:D_0402_1005Metric"
 			(at 63.5 97.79 0)
 			(effects
@@
 			)
 		)
-		(property "Footprint" "PCM_Diode_SMD_AKL:D_0402_1005Metric"
+		(property "Footprint" "Diode_SMD:D_0402_1005Metric"
 			(at 71.12 97.79 0)
 			(effects

Commit message: Bump versions
Parts:
- renumbered J402 to J401, J401 to J402
Changed lines of the file:
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@@
 	(title_block
 		(title "Hat Labs Serial Interface Device (HALSER)")
-		(date "2024-11-20")
-		(rev "1.0.0-a1")
+		(date "2024-12-20")
+		(rev "1.0.0")
 		(company "Hat Labs oy")
 		(comment 1 "https://creativecommons.org/licenses/by-sa/4.0")
@@
 		(on_board yes)
 		(dnp no)
-		(property "Reference" "J401"
+		(property "Reference" "J402"
 			(at 43.9928 77.0382 0)
 			(effects
@@
 			(project "HALMET"
 				(path "/dff502f1-2fe5-4c09-a767-aabc78c2e052/00000000-0000-0000-0000-00005f9be197"
-					(reference "J401")
+					(reference "J402")
 					(unit 1)
 				)
@@
 		(on_board yes)
 		(dnp no)
-		(property "Reference" "J402"
+		(property "Reference" "J401"
 			(at 43.9928 61.7982 0)
 			(effects
@@
 			(project "HALSER"
 				(path "/dff502f1-2fe5-4c09-a767-aabc78c2e052/00000000-0000-0000-0000-00005f9be197"
-					(reference "J402")
+					(reference "J401")
 					(unit 1)
 				)
