File: PCB.kicad_sch (KiCad schematic)
At the start: 8 parts

Commit message: Redo schematics
Parts:
- added H603, H604: MountingHole, HALMET:MountingSlot_3.2mm_M3_Unplated, symbol Mechanical:MountingHole
- renumbered H1001 to H601, H1002 to H602

Commit message: WIP wiring
Parts:
- G501: footprint HALMET:cc-by_5mm -> HALSER:cc-by_5mm
- G505: footprint HALMET:Hat_Labs_25.4mm -> HALSER:Hat_Labs_25.4mm
- G505: footprint HALMET:HaL_picto_8mm -> HALSER:HaL_picto_8mm
- H601, H602, H603, H604: footprint HALMET:MountingSlot_3.2mm_M3_Unplated -> MountingHole:MountingHole_3.2mm_M3_ISO7380
Changed lines of the file:
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@@
 			)
 		)
-		(property "Footprint" "HALMET:MountingSlot_3.2mm_M3_Unplated"
+		(property "Footprint" "MountingHole:MountingHole_3.2mm_M3_ISO7380"
 			(at 48.26 46.99 0)
 			(effects
@@
 		)
 		(property "Sim.Pins" ""
+			(at 48.26 46.99 0)
+			(effects
+				(font
+					(size 1.27 1.27)
+				)
+				(hide yes)
+			)
+		)
+		(property "Note" ""
 			(at 48.26 46.99 0)
 			(effects
@@
 			)
 		)
-		(property "Footprint" "HALMET:MountingSlot_3.2mm_M3_Unplated"
+		(property "Footprint" "MountingHole:MountingHole_3.2mm_M3_ISO7380"
 			(at 48.26 54.61 0)
 			(effects
@@
 		)
 		(property "Sim.Pins" ""
+			(at 48.26 54.61 0)
+			(effects
+				(font
+					(size 1.27 1.27)
+				)
+				(hide yes)
+			)
+		)
+		(property "Note" ""
 			(at 48.26 54.61 0)
 			(effects
@@
 			)
 		)
+		(property "Note" ""
+			(at 160.02 55.88 0)
+			(effects
+				(font
+					(size 1.27 1.27)
+				)
+				(hide yes)
+			)
+		)
 		(instances
 			(project "HALMET"
@@
 			)
 		)
-		(property "Footprint" "HALMET:MountingSlot_3.2mm_M3_Unplated"
+		(property "Footprint" "MountingHole:MountingHole_3.2mm_M3_ISO7380"
 			(at 48.26 62.23 0)
 			(effects
@@
 		)
 		(property "Sim.Pins" ""
+			(at 48.26 62.23 0)
+			(effects
+				(font
+					(size 1.27 1.27)
+				)
+				(hide yes)
+			)
+		)
+		(property "Note" ""
 			(at 48.26 62.23 0)
 			(effects
@@
 			)
 		)
-		(property "Footprint" "HALMET:cc-by_5mm"
+		(property "Footprint" "HALSER:cc-by_5mm"
 			(at 160.02 46.99 0)
 			(effects
@@
 		)
 		(property "Sim.Pins" ""
+			(at 160.02 46.99 0)
+			(effects
+				(font
+					(size 1.27 1.27)
+				)
+				(hide yes)
+			)
+		)
+		(property "Note" ""
 			(at 160.02 46.99 0)
 			(effects
@@
 			)
 		)
-		(property "Footprint" "HALMET:Hat_Labs_25.4mm"
+		(property "Footprint" "HALSER:Hat_Labs_25.4mm"
 			(at 160.02 82.55 0)
 			(effects
@@
 		)
 		(property "Sim.Pins" ""
+			(at 160.02 82.55 0)
+			(effects
+				(font
+					(size 1.27 1.27)
+				)
+				(hide yes)
+			)
+		)
+		(property "Note" ""
 			(at 160.02 82.55 0)
 			(effects
@@
 			)
 		)
-		(property "Footprint" "HALMET:MountingSlot_3.2mm_M3_Unplated"
+		(property "Footprint" "MountingHole:MountingHole_3.2mm_M3_ISO7380"
 			(at 48.26 69.85 0)
 			(effects
@@
 		)
 		(property "Sim.Pins" ""
+			(at 48.26 69.85 0)
+			(effects
+				(font
+					(size 1.27 1.27)
+				)
+				(hide yes)
+			)
+		)
+		(property "Note" ""
 			(at 48.26 69.85 0)
 			(effects
@@
 		(exclude_from_sim yes)
 		(in_bom no)
-		(on_board no)
+		(on_board yes)
 		(dnp no)
 		(fields_autoplaced yes)
@@
 		)
 		(property "Sim.Pins" ""
+			(at 160.02 64.77 0)
+			(effects
+				(font
+					(size 1.27 1.27)
+				)
+				(hide yes)
+			)
+		)
+		(property "Note" ""
 			(at 160.02 64.77 0)
 			(effects
@@
 			)
 		)
-		(property "Footprint" "HALMET:HaL_picto_8mm"
+		(property "Footprint" "HALSER:HaL_picto_8mm"
 			(at 160.02 91.44 0)
 			(effects
@@
 		)
 		(property "Sim.Pins" ""
+			(at 160.02 91.44 0)
+			(effects
+				(font
+					(size 1.27 1.27)
+				)
+				(hide yes)
+			)
+		)
+		(property "Note" ""
 			(at 160.02 91.44 0)
 			(effects
@@
 			(at 160.02 73.66 0)
 			(effects
+				(font
+					(size 1.27 1.27)
+				)
+				(hide yes)
+			)
+		)
+		(property "Note" ""
+			(at 160.02 73.66 0)
+			(effects

Commit message: Fix issues found in -a1
Other:
- company: Hat Labs Ltd -> Hat Labs oy
- title: Hat Labs Marine Engine & Tank interface (HALMET) -> Hat Labs Serial Interface Device (HALSER)
Changed lines of the file:
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@@
 	(paper "A4")
 	(title_block
-		(title "Hat Labs Marine Engine & Tank interface (HALMET)")
-		(date "2024-01-18")
-		(rev "1.0.1")
-		(company "Hat Labs Ltd")
+		(title "Hat Labs Serial Interface Device (HALSER)")
+		(date "2024-11-20")
+		(rev "1.0.0-a1")
+		(company "Hat Labs oy")
 		(comment 1 "https://creativecommons.org/licenses/by-sa/4.0")
 		(comment 2 "To view a copy of this license, visit ")
@@
 		(exclude_from_sim yes)
 		(in_bom no)
-		(on_board yes)
+		(on_board no)
 		(dnp no)
 		(fields_autoplaced yes)
