File: USB.kicad_sch (KiCad schematic)
At the start: 16 parts, among them J401 USB_B_Micro, Q401 S8050, Q402 S8050, U401 CH340C

Commit message: Redo schematics
Parts:
- removed C1002: 100nF, Capacitor_SMD:C_0402_1005Metric, symbol Device:C
- removed C403, C404: 10pF/50V, Capacitor_SMD:C_0402_1005Metric, symbol Device:C
- removed J401: USB_B_Micro, Connector_USB:USB_Micro-B_Wuerth_614105150721_Vertical, symbol HALMET:USB_B_Micro-Connector
- removed Q401, Q402: S8050, Package_TO_SOT_SMD:SOT-23, symbol HALMET:S8050
- removed R401, R402: 10k, Resistor_SMD:R_0402_1005Metric, symbol Device:R
- removed U401: CH340C, Package_SO:SOIC-16_3.9x9.9mm_P1.27mm, symbol Interface_USB:CH340C
- added J802: USB_C_Receptacle_USB2.0_16P, HALSER:Shou Han Type-C 16P LTH6.8, symbol Connector:USB_C_Receptacle_USB2.0_16P
- added R801, R802: 5.1k, PCM_Resistor_SMD_AKL:R_0402_1005Metric, symbol Device:R
- C801: renamed from C503; footprint Capacitor_SMD:C_0805_2012Metric -> PCM_Capacitor_SMD_AKL:C_0603_1608Metric; LCSC C28323 -> C15849
- C802: renamed from C402; footprint Capacitor_SMD:C_0603_1608Metric -> PCM_Capacitor_SMD_AKL:C_0603_1608Metric
- D801: renamed from D903; footprint Diode_SMD:D_0402_1005Metric -> PCM_Diode_SMD_AKL:D_0402_1005Metric
- D802: renamed from D904; footprint Diode_SMD:D_0402_1005Metric -> PCM_Diode_SMD_AKL:D_0402_1005Metric
- D803: renamed from D905; footprint Diode_SMD:D_0402_1005Metric -> PCM_Diode_SMD_AKL:D_0402_1005Metric
- F801: renamed from F401; footprint Fuse:Fuse_1206_3216Metric -> PCM_Fuse_AKL:Fuse_1206_3216Metric
- FB801: renamed from FB401; footprint Inductor_SMD:L_0805_2012Metric -> PCM_Ferrite_SMD_AKL:Ferrite_0805_2012Metric
Connections:
- net GND: now also J802.A1 (GND), J802.A12 (GND), J802.B1 (GND), J802.B12 (GND), J802.S1 (SHIELD), R801.2, R802.2
- net USB_D+: now also D803.2 (A2), J802.A6 (D+), J802.B6 (D+); no longer D802.2 (A2)
- net USB_D-: now also D802.2 (A2), J802.A7 (D-), J802.B7 (D-); no longer D803.2 (A2)
- net VBUS: now also J802.A4 (VBUS), J802.A9 (VBUS), J802.B4 (VBUS), J802.B9 (VBUS)
- new net: J802.A5 (CC1), R802.1
- new net: J802.B5 (CC2), R801.1
- no-connect marks 6 -> 2
Other:
- note removed: "C403 and C404 are virtual for now"
- moved on the sheet: C801, C802, D801, D802, D803, F801, FB801

Commit message: Further design adjustments
Connections:
- net CC1: now reaches J802.A5 (CC1), R802.1
- net CC2: now reaches J802.B5 (CC2), R801.1
Changed lines of the file:
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@@
+		)
+	)
+	(label "CC1"
+		(at 72.39 49.53 0)
+		(fields_autoplaced yes)
+		(effects
+			(font
+				(size 1.27 1.27)
+			)
+			(justify left bottom)
 		)
 	)
@@
 		(fields_autoplaced yes)
 		(effects
+			(font
+				(size 1.27 1.27)
+			)
+			(justify left bottom)
+		)
+	)
+	(label "CC2"
+		(at 72.39 52.07 0)
+		(fields_autoplaced yes)
+		(effects

Commit message: Fix issues found in -a1
Parts:
- C801, C802: footprint PCM_Capacitor_SMD_AKL:C_0603_1608Metric -> Capacitor_SMD:C_0603_1608Metric
- D801, D802, D803: footprint PCM_Diode_SMD_AKL:D_0402_1005Metric -> Diode_SMD:D_0402_1005Metric
- F801: footprint PCM_Fuse_AKL:Fuse_1206_3216Metric -> Fuse:Fuse_1206_3216Metric
- FB801: footprint PCM_Ferrite_SMD_AKL:Ferrite_0805_2012Metric -> Inductor_SMD:L_0805_2012Metric
- R801, R802: footprint PCM_Resistor_SMD_AKL:R_0402_1005Metric -> Resistor_SMD:R_0402_1005Metric
Other:
- company: Hat Labs Ltd -> Hat Labs oy
- title: Hat Labs Marine Engine & Tank interface (HALMET) -> Hat Labs Serial Interface Device (HALSER)
Changed lines of the file:
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@@
 	(paper "A4")
 	(title_block
-		(title "Hat Labs Marine Engine & Tank interface (HALMET)")
-		(date "2024-01-18")
-		(rev "1.0.1")
-		(company "Hat Labs Ltd")
+		(title "Hat Labs Serial Interface Device (HALSER)")
+		(date "2024-11-20")
+		(rev "1.0.0-a1")
+		(company "Hat Labs oy")
 		(comment 1 "https://creativecommons.org/licenses/by-sa/4.0")
 		(comment 2 "To view a copy of this license, visit ")
@@
 			)
 		)
-		(property "Footprint" "PCM_Capacitor_SMD_AKL:C_0603_1608Metric"
+		(property "Footprint" "Capacitor_SMD:C_0603_1608Metric"
 			(at 197.8152 52.07 0)
 			(effects
@@
 			)
 		)
-		(property "Footprint" "PCM_Ferrite_SMD_AKL:Ferrite_0805_2012Metric"
+		(property "Footprint" "Inductor_SMD:L_0805_2012Metric"
 			(at 107.95 42.672 90)
 			(effects
@@
 			)
 		)
-		(property "Footprint" "PCM_Fuse_AKL:Fuse_1206_3216Metric"
+		(property "Footprint" "Fuse:Fuse_1206_3216Metric"
 			(at 88.9 42.672 90)
 			(effects
@@
 			)
 		)
-		(property "Footprint" "PCM_Capacitor_SMD_AKL:C_0603_1608Metric"
+		(property "Footprint" "Capacitor_SMD:C_0603_1608Metric"
 			(at 101.2952 63.5 0)
 			(effects
@@
 			)
 		)
-		(property "Footprint" "PCM_Resistor_SMD_AKL:R_0402_1005Metric"
+		(property "Footprint" "Resistor_SMD:R_0402_1005Metric"
 			(at 76.962 72.39 90)
 			(effects
@@
 			)
 		)
-		(property "Footprint" "PCM_Diode_SMD_AKL:D_0402_1005Metric"
+		(property "Footprint" "Diode_SMD:D_0402_1005Metric"
 			(at 132.08 59.69 0)
 			(effects
@@
 			)
 		)
-		(property "Footprint" "PCM_Resistor_SMD_AKL:R_0402_1005Metric"
+		(property "Footprint" "Resistor_SMD:R_0402_1005Metric"
 			(at 76.708 72.39 90)
 			(effects
@@
 			)
 		)
-		(property "Footprint" "PCM_Diode_SMD_AKL:D_0402_1005Metric"
+		(property "Footprint" "Diode_SMD:D_0402_1005Metric"
 			(at 138.43 66.04 0)
 			(effects
@@
 			)
 		)
-		(property "Footprint" "PCM_Diode_SMD_AKL:D_0402_1005Metric"
+		(property "Footprint" "Diode_SMD:D_0402_1005Metric"
 			(at 125.73 55.88 0)
 			(effects

Commit message: Bump versions
Parts:
- renumbered J802 to J801
Changed lines of the file:
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@@
 	(title_block
 		(title "Hat Labs Serial Interface Device (HALSER)")
-		(date "2024-11-20")
-		(rev "1.0.0-a1")
+		(date "2024-12-20")
+		(rev "1.0.0")
 		(company "Hat Labs oy")
 		(comment 1 "https://creativecommons.org/licenses/by-sa/4.0")
@@
 		(dnp no)
 		(fields_autoplaced yes)
-		(property "Reference" "J802"
+		(property "Reference" "J801"
 			(at 52.07 36.83 0)
 			(effects
@@
 			(project ""
 				(path "/dff502f1-2fe5-4c09-a767-aabc78c2e052/00000000-0000-0000-0000-00005f89c30a"
-					(reference "J802")
+					(reference "J801")
 					(unit 1)
 				)
