File: canbus.kicad_sch (KiCad schematic)
At the start: 7 parts, among them U501 SN65HVD230DR

Commit message: Redo schematics
Parts:
- added C201, C202: 100pF, PCM_Capacitor_SMD_AKL:C_0603_1608Metric, symbol Device:C_Small
- added D201: SM24CANB, PCM_Package_TO_SOT_SMD_AKL:SOT-23, symbol Diode:SM712_SOT23
- added FL201: PCAQ2012B-201T030, PCM_Ferrite_SMD_AKL:Ferrite_0805_2012Metric, symbol Device:Filter_EMI_CommonMode
- C203: renamed from C602; footprint Capacitor_SMD:C_0402_1005Metric -> PCM_Capacitor_SMD_AKL:C_0402_1005Metric
- R201: renamed from R601; footprint Resistor_SMD:R_0805_2012Metric -> PCM_Resistor_SMD_AKL:R_0805_2012Metric
- R202: renamed from R602; footprint Resistor_SMD:R_0805_2012Metric -> PCM_Resistor_SMD_AKL:R_0805_2012Metric
- R203: renamed from R503; footprint Resistor_SMD:R_0402_1005Metric -> PCM_Resistor_SMD_AKL:R_0402_1005Metric
- R204: renamed from R213; footprint Resistor_SMD:R_0402_1005Metric -> PCM_Resistor_SMD_AKL:R_0402_1005Metric
- U201: renamed from U501; footprint Package_SO:SOIC-8_3.9x4.9mm_P1.27mm -> PCM_Package_SO_AKL:SOIC-8_3.9x4.9mm_P1.27mm
- renumbered JP601 to JP201
Connections:
- net CAN_H: now also FL201.1; no longer U201.7 (CANH)
- net CAN_L: now also FL201.3; no longer U201.6 (CANL)
- net GND: now also C201.2, C202.2, D201.3 (common)
- new net: C202.1, D201.2 (A2), FL201.4, U201.6 (CANL)
- new net: C201.1, D201.1 (A1), FL201.2, U201.7 (CANH)
Other:
- moved on the sheet: JP201, R201, R202

Commit message: WIP wiring
Parts:
- removed JP201: SolderJumper_2_Open, HALMET:SolderJumper-2_P1.3mm_Open_TrianglePad_Narrow, symbol Jumper:SolderJumper_2_Open
- removed R201, R202: 240R, PCM_Resistor_SMD_AKL:R_0805_2012Metric, symbol Device:R
- FL201: footprint PCM_Ferrite_SMD_AKL:Ferrite_0805_2012Metric -> HALSER:L_CommonModeChoke_PCAQ2012B; symbol Device:Filter_EMI_CommonMode -> Device:L_Ferrite_Coupled_1243
Connections:
- net CAN_L: now also FL201.4; no longer FL201.3
- net at C202.1, U201.6 (CANL): now also D201.1 (A1), FL201.3; no longer D201.2 (A2), FL201.4
- net at C201.1, FL201.2, U201.7 (CANH): now also D201.2 (A2); no longer D201.1 (A1)
Other:
- note removed: "Optional termination resistance for the bus"

Commit message: Fix issues found in -a1
Parts:
- C201, C202: footprint PCM_Capacitor_SMD_AKL:C_0603_1608Metric -> Capacitor_SMD:C_0603_1608Metric
- C203: footprint PCM_Capacitor_SMD_AKL:C_0402_1005Metric -> Capacitor_SMD:C_0402_1005Metric
- D201: footprint PCM_Package_TO_SOT_SMD_AKL:SOT-23 -> Package_TO_SOT_SMD:SOT-23
- R203, R204: footprint PCM_Resistor_SMD_AKL:R_0402_1005Metric -> Resistor_SMD:R_0402_1005Metric
- U201: footprint PCM_Package_SO_AKL:SOIC-8_3.9x4.9mm_P1.27mm -> Package_SO:SOIC-8_3.9x4.9mm_P1.27mm
Other:
- company: Hat Labs Ltd -> Hat Labs oy
- title: Hat Labs Marine Engine & Tank interface (HALMET) -> Hat Labs Serial Interface Device (HALSER)
Changed lines of the file:
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@@
 	(paper "A4")
 	(title_block
-		(title "Hat Labs Marine Engine & Tank interface (HALMET)")
-		(date "2024-01-18")
-		(rev "1.0.1")
-		(company "Hat Labs Ltd")
+		(title "Hat Labs Serial Interface Device (HALSER)")
+		(date "2024-11-20")
+		(rev "1.0.0-a1")
+		(company "Hat Labs oy")
 		(comment 1 "https://creativecommons.org/licenses/by-sa/4.0")
 		(comment 2 "To view a copy of this license, visit ")
@@
 			)
 		)
-		(property "Footprint" "PCM_Capacitor_SMD_AKL:C_0402_1005Metric"
+		(property "Footprint" "Capacitor_SMD:C_0402_1005Metric"
 			(at 127.3048 99.06 0)
 			(effects
@@
 			)
 		)
-		(property "Footprint" "PCM_Package_SO_AKL:SOIC-8_3.9x4.9mm_P1.27mm"
+		(property "Footprint" "Package_SO:SOIC-8_3.9x4.9mm_P1.27mm"
 			(at 134.62 123.19 0)
 			(effects
@@
 			)
 		)
-		(property "Footprint" "PCM_Resistor_SMD_AKL:R_0402_1005Metric"
+		(property "Footprint" "Resistor_SMD:R_0402_1005Metric"
 			(at 147.32 119.38 0)
 			(effects
@@
 			)
 		)
-		(property "Footprint" "PCM_Resistor_SMD_AKL:R_0402_1005Metric"
+		(property "Footprint" "Resistor_SMD:R_0402_1005Metric"
 			(at 189.23 101.6 0)
 			(effects
@@
 			)
 		)
-		(property "Footprint" "PCM_Capacitor_SMD_AKL:C_0603_1608Metric"
+		(property "Footprint" "Capacitor_SMD:C_0603_1608Metric"
 			(at 83.82 120.65 0)
 			(effects
@@
 			)
 		)
-		(property "Footprint" "PCM_Package_TO_SOT_SMD_AKL:SOT-23"
+		(property "Footprint" "Package_TO_SOT_SMD:SOT-23"
 			(at 110.49 129.54 0)
 			(effects
@@
 			)
 		)
-		(property "Footprint" "PCM_Capacitor_SMD_AKL:C_0603_1608Metric"
+		(property "Footprint" "Capacitor_SMD:C_0603_1608Metric"
 			(at 88.9 120.65 0)
 			(effects

Commit message: Bump versions
Parts:
- renumbered R203 to R201, R204 to R202
Changed lines of the file:
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@@
 	(title_block
 		(title "Hat Labs Serial Interface Device (HALSER)")
-		(date "2024-11-20")
-		(rev "1.0.0-a1")
+		(date "2024-12-20")
+		(rev "1.0.0")
 		(company "Hat Labs oy")
 		(comment 1 "https://creativecommons.org/licenses/by-sa/4.0")
@@
 		(on_board yes)
 		(dnp no)
-		(property "Reference" "R203"
+		(property "Reference" "R201"
 			(at 148.8186 118.2116 0)
 			(effects
@@
 			(project "HALMET"
 				(path "/dff502f1-2fe5-4c09-a767-aabc78c2e052/00000000-0000-0000-0000-00005f733ba4"
-					(reference "R203")
+					(reference "R201")
 					(unit 1)
 				)
@@
 		(dnp no)
 		(fields_autoplaced yes)
-		(property "Reference" "R204"
+		(property "Reference" "R202"
 			(at 191.77 100.3299 0)
 			(effects
@@
 			(project "HALMET"
 				(path "/dff502f1-2fe5-4c09-a767-aabc78c2e052/00000000-0000-0000-0000-00005f733ba4"
-					(reference "R204")
+					(reference "R202")
 					(unit 1)
 				)
