File: onewire.kicad_sch (KiCad schematic)
At the start: 9 parts, among them J801 Conn_01x03

Commit message: Redo schematics
Parts:
- C501: renamed from C803; footprint Capacitor_SMD:C_1206_3216Metric -> PCM_Capacitor_SMD_AKL:C_1206_3216Metric
- C502: renamed from C802; footprint Capacitor_SMD:C_0603_1608Metric -> PCM_Capacitor_SMD_AKL:C_0603_1608Metric
- C503: renamed from C801; footprint Capacitor_SMD:C_0402_1005Metric -> PCM_Capacitor_SMD_AKL:C_0603_1608Metric; LCSC C15525 -> C19702
- D501: renamed from D503; footprint Diode_SMD:D_0402_1005Metric -> PCM_Diode_SMD_AKL:D_0402_1005Metric
- D502: renamed from D504; footprint Diode_SMD:D_0402_1005Metric -> PCM_Diode_SMD_AKL:D_0402_1005Metric
- FB501: renamed from FB801; footprint Inductor_SMD:L_0805_2012Metric -> PCM_Ferrite_SMD_AKL:Ferrite_0805_2012Metric
- J501: renamed from J801; value Conn_01x03 -> 1-Wire Male Header
- R501: renamed from R801; footprint Resistor_SMD:R_0402_1005Metric -> PCM_Resistor_SMD_AKL:R_0402_1005Metric
- R502: renamed from R802; footprint Resistor_SMD:R_0805_2012Metric -> PCM_Resistor_SMD_AKL:R_0805_2012Metric

Commit message: Further design adjustments
Connections:
- net DQ_CONN: no longer D501.2 (A2), R502.2
- new net DQ_C: D501.2 (A2), R502.2
Changed lines of the file:
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@@
 		)
 	)
-	(label "DQ_CONN"
+	(label "DQ_C"
 		(at 104.14 59.69 180)
 		(fields_autoplaced yes)
@@
 		)
 	)
-	(label "DQ_CONN"
-		(at 41.91 92.71 180)
-		(fields_autoplaced yes)
-		(effects
-			(font
-				(size 1.27 1.27)
-			)
-			(justify right bottom)
-		)
-	)
 	(hierarchical_label "DQ"
 		(shape input)
@@
 		)
 	)
+	(hierarchical_label "DQ_C"
+		(shape input)
+		(at 41.91 92.71 180)
+		(fields_autoplaced yes)
+		(effects
+			(font
+				(size 1.27 1.27)
+			)
+			(justify right)
+		)
+	)

Commit message: Further manufacturing tweaks
Connections:
- net DQ_CONN is gone; now on net DQ_C: J501.3 (Pin_3)
Changed lines of the file:
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@@
 		)
 	)
-	(label "DQ_CONN"
+	(label "DQ_C"
 		(at 45.72 59.69 0)
 		(fields_autoplaced yes)

Commit message: Fix issues found in -a1
Parts:
- C501: footprint PCM_Capacitor_SMD_AKL:C_1206_3216Metric -> Capacitor_SMD:C_1206_3216Metric
- C502, C503: footprint PCM_Capacitor_SMD_AKL:C_0603_1608Metric -> Capacitor_SMD:C_0603_1608Metric
- D501, D502: footprint PCM_Diode_SMD_AKL:D_0402_1005Metric -> Diode_SMD:D_0402_1005Metric
- FB501: footprint PCM_Ferrite_SMD_AKL:Ferrite_0805_2012Metric -> Inductor_SMD:L_0805_2012Metric
- R501: footprint PCM_Resistor_SMD_AKL:R_0402_1005Metric -> Resistor_SMD:R_0402_1005Metric
- R502: footprint PCM_Resistor_SMD_AKL:R_0805_2012Metric -> Resistor_SMD:R_0805_2012Metric
Other:
- company: Hat Labs Ltd -> Hat Labs oy
- title: Hat Labs Marine Engine & Tank interface (HALMET) -> Hat Labs Serial Interface Device (HALSER)
Changed lines of the file:
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@@
 	(paper "A4")
 	(title_block
-		(title "Hat Labs Marine Engine & Tank interface (HALMET)")
-		(date "2024-01-18")
-		(rev "1.0.1")
-		(company "Hat Labs Ltd")
+		(title "Hat Labs Serial Interface Device (HALSER)")
+		(date "2024-11-20")
+		(rev "1.0.0-a1")
+		(company "Hat Labs oy")
 		(comment 1 "https://creativecommons.org/licenses/by-sa/4.0")
 		(comment 2 "To view a copy of this license, visit ")
@@
 			)
 		)
-		(property "Footprint" "PCM_Resistor_SMD_AKL:R_0402_1005Metric"
+		(property "Footprint" "Resistor_SMD:R_0402_1005Metric"
 			(at 111.76 38.862 90)
 			(effects
@@
 			)
 		)
-		(property "Footprint" "PCM_Capacitor_SMD_AKL:C_1206_3216Metric"
+		(property "Footprint" "Capacitor_SMD:C_1206_3216Metric"
 			(at 112.0648 106.68 0)
 			(effects
@@
 			)
 		)
-		(property "Footprint" "PCM_Capacitor_SMD_AKL:C_0603_1608Metric"
+		(property "Footprint" "Capacitor_SMD:C_0603_1608Metric"
 			(at 124.1552 106.68 0)
 			(effects
@@
 			)
 		)
-		(property "Footprint" "PCM_Ferrite_SMD_AKL:Ferrite_0805_2012Metric"
+		(property "Footprint" "Inductor_SMD:L_0805_2012Metric"
 			(at 118.11 97.282 90)
 			(effects
@@
 			)
 		)
-		(property "Footprint" "PCM_Resistor_SMD_AKL:R_0805_2012Metric"
+		(property "Footprint" "Resistor_SMD:R_0805_2012Metric"
 			(at 111.76 57.912 90)
 			(effects
@@
 			)
 		)
-		(property "Footprint" "PCM_Capacitor_SMD_AKL:C_0603_1608Metric"
+		(property "Footprint" "Capacitor_SMD:C_0603_1608Metric"
 			(at 117.8052 68.58 0)
 			(effects
@@
 			)
 		)
-		(property "Footprint" "PCM_Diode_SMD_AKL:D_0402_1005Metric"
+		(property "Footprint" "Diode_SMD:D_0402_1005Metric"
 			(at 59.69 105.41 0)
 			(effects
@@
 			)
 		)
-		(property "Footprint" "PCM_Diode_SMD_AKL:D_0402_1005Metric"
+		(property "Footprint" "Diode_SMD:D_0402_1005Metric"
 			(at 53.34 105.41 0)
 			(effects
