File: power-input.kicad_sch (KiCad schematic)
At the start: 23 parts, among them J601 Conn_01x04, U202 XL1509-3.3

Commit message: Redo schematics
Parts:
- removed C304: 47uF/6.3V, Capacitor_SMD:C_1206_3216Metric, symbol Device:C
- removed C707, C710, C711, C712, C714: 10uF/50V, Capacitor_SMD:C_1206_3216Metric, symbol Device:C
- removed C713: 4.7nF/50V, Capacitor_SMD:C_0402_1005Metric, symbol Device:C
- removed C715: 1uF/50V, Capacitor_SMD:C_0805_2012Metric, symbol Device:C
- removed C716: 4.7uF/50V, Capacitor_SMD:C_1206_3216Metric, symbol Device:C
- removed D202: SM24CANB, Package_TO_SOT_SMD:SOT-23, symbol Device:D_TVS_Dual_AAC
- removed D701: B5819W, Diode_SMD:D_SOD-123, symbol Device:D_Schottky
- removed FB704: GZ2012D601TF, Inductor_SMD:L_0805_2012Metric, symbol Device:FerriteBead
- removed J601: Conn_01x04, Connector_Phoenix_MC:PhoenixContact_MCV_1,5_4-G-3.81_1x04_P3.81mm_Vertical, symbol Connector_Generic:Conn_01x04
- removed R703: 4.7R, Resistor_SMD:R_0603_1608Metric, symbol Device:R
- removed U202: XL1509-3.3, Package_SO:SOP-8_3.9x4.9mm_P1.27mm, symbol HALMET:XL1509-ADJE1
- added C701, C703, C704, C705: 10uF/50V, PCM_Capacitor_SMD_AKL:C_1206_3216Metric, symbol Device:C
- added C702: 4.7uF/50V, PCM_Capacitor_SMD_AKL:C_0805_2012Metric, symbol Device:C
- added C706: 100nF/50V, PCM_Capacitor_SMD_AKL:C_0603_1608Metric, symbol Device:C_Small
- added C707: 100nF/16V, PCM_Capacitor_SMD_AKL:C_0402_1005Metric, symbol Device:C_Small
- added J701: CAN Socket, Connector_Phoenix_MC:PhoenixContact_MCV_1,5_4-G-3.81_1x04_P3.81mm_Vertical, symbol Connector_Generic:Conn_01x04
- added R701: 0.1R, PCM_Resistor_SMD_AKL:R_0603_1608Metric, symbol Device:R
- added R702: 75k, PCM_Resistor_SMD_AKL:R_0402_1005Metric, symbol Device:R_Small
- added R703: 24k, PCM_Resistor_SMD_AKL:R_0402_1005Metric, symbol Device:R_Small
- added U701: LMR54410DBVR, SOT-23-6-DBV_TEX, symbol HALSER:LMR54410DBVR
- C708, C709: value 10uF/50V -> 47uF/6.3V; footprint Capacitor_SMD:C_1206_3216Metric -> PCM_Capacitor_SMD_AKL:C_0805_2012Metric; LCSC C13585 -> C16780; Notes 50V -> Min 6.3V
- D701: renamed from D201; footprint Diode_SMD:D_SOD-123 -> PCM_Diode_SMD_AKL:D_SOD-123
- D702: renamed from D301; footprint Diode_SMD:D_SMB -> PCM_Diode_SMD_AKL:D_SMB_TVS
- D703: renamed from D303; footprint Diode_SMD:D_SOD-123 -> PCM_Diode_SMD_AKL:D_SOD-123
- F701: renamed from F301; footprint Fuse:Fuse_1812_4532Metric -> PCM_Fuse_AKL:Fuse_1812_4532Metric
- L701: value NLCV32T-100K-EFR -> CBC3225T100KR; LCSC C295195 -> C90321; Notes Alternative: CBC3225T100KR -> Alternatives: CBC3225T100KR, CBC3225T100MR, NLCV32T-100K-PFR
- L702: renamed from L301; value SMMS0650-470M -> SLO0530H6R8MTT; footprint HALMET:SMMS0650-1R0M -> Inductor_SMD:L_Chilisin_BMRA00050530; LCSC C149588 -> C325965
Connections:
- net CAN_H: now also J701.3 (Pin_3)
- net CAN_L: now also J701.4 (Pin_4)
- net GND: now also C701.2, C702.1, C705.2, C706.2, J701.1 (Pin_1), R701.1, R703.2, U701.2 (GND)
- net IN: now also L701.2, C702.2, C703.1, C704.1, C705.1, C706.1, U701.4 (EN), U701.5 (VIN); no longer C708.1, C709.1
- net SW: now also C707.1, U701.6 (SW)
- net Vin_protected: now also C701.1
- net +3.3V renamed +3V3
- net +3V3: now also C708.1, C709.1, R702.1
- net CAN_+ renamed Vin
- net Vin: now also J701.2 (Pin_2)
- new net: C703.2, C704.2, R701.2
- new net CB: C707.2, U701.1 (CB)
- new net FB: R702.2, R703.1, U701.3 (FB)
Other:
- note added: "Converter IC voltage range 4.5-50V, however, Vin needs to be a bit higher to give some headroom for the PTC fuse."
- note added: "Input filter for limiting conducted noise emissions at power input lines."
- note removed: "Bulk input capacitance is implemented with a number of 10uF MLCC caps to manage the cost."
- note removed: "Converter IC voltage range 4.5-50V, however, Vin needs to be a bit higher to give some headroom for the PTC fuse and polarity protection diode."
- note removed: "First stage HF input filter. Design as per TI SNVA886."
- note removed: "NMEA 2000"
- note removed: "Second stage input filter for limiting conducted noise emissions at power input lines. Design as per Rohm 62AN101E."
- company: Hat Labs Ltd -> Hat Labs Oy
- title: Hat Labs Marine Engine & Tank interface (HALMET) -> SH-ESP32
- moved on the sheet: D701, L702

Commit message: WIP wiring
Parts:
- U701: footprint SOT-23-6-DBV_TEX -> PCM_Package_TO_SOT_SMD_AKL:SOT-23-6
Connections:
- net +3V3 renamed +3.3V
Changed lines of the file:
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@@
 	)
 	(junction
-		(at 252.73 107.95)
-		(diameter 0)
-		(color 0 0 0 0)
-	)
-	(junction
 		(at 170.18 102.87)
 		(diameter 0)
@@
 	(wire
 		(pts
-			(xy 250.19 107.95) (xy 252.73 107.95)
-		)
-		(stroke
-			(width 0)
-			(type default)
-		)
-	)
-	(wire
-		(pts
 			(xy 59.69 85.09) (xy 59.69 102.87)
 		)
@@
 	(wire
 		(pts
-			(xy 252.73 107.95) (xy 261.62 107.95)
+			(xy 250.19 107.95) (xy 261.62 107.95)
 		)
 		(stroke
@@
 			)
 		)
+		(property "Note" ""
+			(at 209.55 107.95 0)
+			(effects
+				(font
+					(size 1.27 1.27)
+				)
+				(hide yes)
+			)
+		)
 		(pin "1"
 		)
@@
 			)
 		)
+		(property "Note" ""
+			(at 97.79 53.34 0)
+			(effects
+				(font
+					(size 1.27 1.27)
+				)
+				(hide yes)
+			)
+		)
 		(pin "1"
 		)
@@
 			)
 		)
-		(property "Value" "+3V3"
+		(property "Value" "+3.3V"
 			(at 262.001 103.5558 0)
 			(effects
@@
 			)
 		)
+		(property "Note" ""
+			(at 44.45 53.34 0)
+			(effects
+				(font
+					(size 1.27 1.27)
+				)
+				(hide yes)
+			)
+		)
 		(pin "1"
 		)
@@
 			)
 		)
+		(property "Note" ""
+			(at 137.16 60.96 0)
+			(effects
+				(font
+					(size 1.27 1.27)
+				)
+				(hide yes)
+			)
+		)
 		(pin "1"
 		)
@@
 			)
 		)
+		(property "Note" ""
+			(at 154.94 53.34 0)
+			(effects
+				(font
+					(size 1.27 1.27)
+				)
+				(hide yes)
+			)
+		)
 		(pin "1"
 		)
@@
 			)
 		)
+		(property "Note" ""
+			(at 49.53 85.09 0)
+			(effects
+				(font
+					(size 1.27 1.27)
+				)
+				(hide yes)
+			)
+		)
 		(pin "1"
 		)
@@
 			)
 		)
+		(property "Note" ""
+			(at 127 106.68 0)
+			(effects
+				(font
+					(size 1.27 1.27)
+				)
+				(hide yes)
+			)
+		)
 		(pin "1"
 		)
@@
 			)
 		)
+		(property "Note" ""
+			(at 121.92 116.84 0)
+			(effects
+				(font
+					(size 1.27 1.27)
+				)
+				(hide yes)
+			)
+		)
 		(pin "1"
 		)
@@
 			)
 		)
+		(property "Note" ""
+			(at 95.25 102.87 0)
+			(effects
+				(font
+					(size 1.27 1.27)
+				)
+				(hide yes)
+			)
+		)
 		(pin "1"
 		)
@@
 			)
 		)
+		(property "Note" ""
+			(at 107.95 106.68 0)
+			(effects
+				(font
+					(size 1.27 1.27)
+				)
+				(hide yes)
+			)
+		)
 		(pin "1"
 		)
@@
 			)
 		)
+		(property "Note" ""
+			(at 222.25 113.03 0)
+			(effects
+				(font
+					(size 1.27 1.27)
+				)
+				(hide yes)
+			)
+		)
 		(pin "1"
 		)
@@
 			)
 		)
+		(property "Note" ""
+			(at 222.25 121.92 0)
+			(effects
+				(font
+					(size 1.27 1.27)
+				)
+				(hide yes)
+			)
+		)
 		(pin "1"
 		)
@@
 			)
 		)
+		(property "Note" ""
+			(at 116.84 106.68 0)
+			(effects
+				(font
+					(size 1.27 1.27)
+				)
+				(hide yes)
+			)
+		)
 		(pin "1"
 		)
@@
 			)
 		)
+		(property "Note" ""
+			(at 86.36 106.68 0)
+			(effects
+				(font
+					(size 1.27 1.27)
+				)
+				(hide yes)
+			)
+		)
 		(pin "1"
 		)
@@
 			)
 		)
+		(property "Note" ""
+			(at 156.21 106.68 0)
+			(effects
+				(font
+					(size 1.27 1.27)
+				)
+				(hide yes)
+			)
+		)
 		(pin "1"
 		)
@@
 			)
 		)
-		(pin "1"
-		)
-		(pin "2"
-		)
-		(instances
-			(project "SH-ESP32"
-				(path "/dff502f1-2fe5-4c09-a767-aabc78c2e052/00000000-0000-0000-0000-00005f6faf6e"
-					(reference "C708")
-					(unit 1)
-				)
-			)
-		)
-	)
-	(symbol
-		(lib_id "power:PWR_FLAG")
-		(at 252.73 107.95 0)
-		(unit 1)
-		(exclude_from_sim no)
-		(in_bom yes)
-		(on_board yes)
-		(dnp no)
-		(fields_autoplaced yes)
-		(property "Reference" "#FLG0704"
-			(at 252.73 106.045 0)
-			(effects
-				(font
-					(size 1.27 1.27)
-				)
-				(hide yes)
-			)
-		)
-		(property "Value" "PWR_FLAG"
-			(at 252.73 102.87 0)
-			(effects
-				(font
-					(size 1.27 1.27)
-				)
-			)
-		)
-		(property "Footprint" ""
-			(at 252.73 107.95 0)
-			(effects
-				(font
-					(size 1.27 1.27)
-				)
-				(hide yes)
-			)
-		)
-		(property "Datasheet" "~"
-			(at 252.73 107.95 0)
-			(effects
-				(font
-					(size 1.27 1.27)
-				)
-				(hide yes)
-			)
-		)
-		(property "Description" "Special symbol for telling ERC where power comes from"
-			(at 252.73 107.95 0)
+		(property "Note" ""
+			(at 243.84 111.76 0)
 			(effects
 				(font
@@
 		(pin "1"
 		)
+		(pin "2"
+		)
 		(instances
-			(project ""
+			(project "SH-ESP32"
 				(path "/dff502f1-2fe5-4c09-a767-aabc78c2e052/00000000-0000-0000-0000-00005f6faf6e"
-					(reference "#FLG0704")
+					(reference "C708")
 					(unit 1)
 				)
@@
 			)
 		)
+		(property "Note" ""
+			(at 170.18 114.3 0)
+			(effects
+				(font
+					(size 1.27 1.27)
+				)
+				(hide yes)
+			)
+		)
 		(pin "1"
 		)
@@
 			)
 		)
+		(property "Note" ""
+			(at 250.19 111.76 0)
+			(effects
+				(font
+					(size 1.27 1.27)
+				)
+				(hide yes)
+			)
+		)
 		(pin "1"
 		)
@@
 			)
 		)
-		(property "Footprint" "SOT-23-6-DBV_TEX"
+		(property "Footprint" "PCM_Package_TO_SOT_SMD_AKL:SOT-23-6"
 			(at 164.846 95.758 0)
 			(effects
@@
 			)
 		)
+		(property "Note" ""
+			(at 185.42 107.95 0)
+			(effects
+				(font
+					(size 1.27 1.27)
+				)
+				(hide yes)
+			)
+		)
 		(pin "6"
 		)
@@
 			(at 200.66 99.06 0)
 			(effects
+				(font
+					(size 1.27 1.27)
+				)
+				(hide yes)
+			)
+		)
+		(property "Note" ""
+			(at 200.66 99.06 0)
+			(effects

Commit message: Further design adjustments
Parts:
- added J702: Vin header, Connector_PinHeader_2.54mm:PinHeader_1x02_P2.54mm_Vertical, symbol Connector_Generic:Conn_01x02
- added J703: CAN Header, Connector_PinHeader_2.54mm:PinHeader_1x04_P2.54mm_Vertical, symbol Connector_Generic:Conn_01x04
Connections:
- net CAN_H: now also J703.3 (Pin_3)
- net CAN_L: now also J703.4 (Pin_4)
- net GND: now also J702.1 (Pin_1), J703.1 (Pin_1)
- net Vin: now also J703.2 (Pin_2)
- net IN renamed VIN
- net VIN: now also J702.2 (Pin_2)

Commit message: Further manufacturing tweaks
Parts:
- J701: JLCPCB_CORRECTION (none) -> 5.715;0;180
- J702: JLCPCB_CORRECTION (none) -> 0;1.27;90; LCSC C492427 -> C492401; now left out of the parts list
- J703: JLCPCB_CORRECTION (none) -> 0;3.81;90
Changed lines of the file:
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@@
 			)
 		)
-		(property "JLCPCB_CORRECTION" ""
+		(property "JLCPCB_CORRECTION" "5.715;0;180"
 			(at 44.45 53.34 0)
 			(effects
@@
 		(unit 1)
 		(exclude_from_sim no)
-		(in_bom yes)
+		(in_bom no)
 		(on_board yes)
 		(dnp no)
@@
 			)
 		)
-		(property "LCSC" "C492427"
+		(property "LCSC" "C492401"
+			(at 157.48 137.16 0)
+			(effects
+				(font
+					(size 1.27 1.27)
+				)
+				(hide yes)
+			)
+		)
+		(property "JLCPCB_CORRECTION" "0;1.27;90"
 			(at 157.48 137.16 0)
 			(effects
@@
 			)
 		)
-		(property "JLCPCB_CORRECTION" ""
+		(property "JLCPCB_CORRECTION" "0;3.81;90"
 			(at 44.45 34.29 0)
 			(effects

Commit message: Fix issues found in -a1
Parts:
- C701, C703, C704, C705: footprint PCM_Capacitor_SMD_AKL:C_1206_3216Metric -> Capacitor_SMD:C_1206_3216Metric
- C702, C708, C709: footprint PCM_Capacitor_SMD_AKL:C_0805_2012Metric -> Capacitor_SMD:C_0805_2012Metric
- C706: footprint PCM_Capacitor_SMD_AKL:C_0603_1608Metric -> Capacitor_SMD:C_0603_1608Metric
- C707: footprint PCM_Capacitor_SMD_AKL:C_0402_1005Metric -> Capacitor_SMD:C_0402_1005Metric
- D701, D703: footprint PCM_Diode_SMD_AKL:D_SOD-123 -> Diode_SMD:D_SOD-123
- D702: footprint PCM_Diode_SMD_AKL:D_SMB_TVS -> Diode_SMD:D_SMB
- F701: footprint PCM_Fuse_AKL:Fuse_1812_4532Metric -> Fuse:Fuse_1812_4532Metric
- R701: footprint PCM_Resistor_SMD_AKL:R_0603_1608Metric -> Resistor_SMD:R_0603_1608Metric
- R702, R703: footprint PCM_Resistor_SMD_AKL:R_0402_1005Metric -> Resistor_SMD:R_0402_1005Metric
- U701: footprint PCM_Package_TO_SOT_SMD_AKL:SOT-23-6 -> Package_TO_SOT_SMD:SOT-23-6
Other:
- company: Hat Labs Oy -> Hat Labs oy
- title: SH-ESP32 -> Hat Labs Serial Interface Device (HALSER)
Changed lines of the file:
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@@
 	(paper "A4")
 	(title_block
-		(title "SH-ESP32")
-		(date "2024-10-16")
-		(rev "2.2.1")
-		(company "Hat Labs Oy")
+		(title "Hat Labs Serial Interface Device (HALSER)")
+		(date "2024-11-20")
+		(rev "1.0.0-a1")
+		(company "Hat Labs oy")
 		(comment 1 "https://creativecommons.org/licenses/by-sa/4.0")
 		(comment 2 "To view a copy of this license, visit ")
-		(comment 3 "SH-ESP32 is licensed under CC BY-SA 4.0.")
+		(comment 3 "HALMET is licensed under CC BY-SA 4.0.")
 	)
 	(junction
@@
 			)
 		)
-		(property "Footprint" "PCM_Fuse_AKL:Fuse_1812_4532Metric"
+		(property "Footprint" "Fuse:Fuse_1812_4532Metric"
 			(at 97.79 51.562 90)
 			(effects
@@
 			)
 		)
-		(property "Footprint" "PCM_Diode_SMD_AKL:D_SMB_TVS"
+		(property "Footprint" "Diode_SMD:D_SMB"
 			(at 137.16 60.96 0)
 			(effects
@@
 			)
 		)
-		(property "Footprint" "PCM_Diode_SMD_AKL:D_SOD-123"
+		(property "Footprint" "Diode_SMD:D_SOD-123"
 			(at 154.94 53.34 0)
 			(effects
@@
 			)
 		)
-		(property "Footprint" "PCM_Diode_SMD_AKL:D_SOD-123"
+		(property "Footprint" "Diode_SMD:D_SOD-123"
 			(at 49.53 85.09 0)
 			(effects
@@
 			)
 		)
-		(property "Footprint" "PCM_Capacitor_SMD_AKL:C_1206_3216Metric"
+		(property "Footprint" "Capacitor_SMD:C_1206_3216Metric"
 			(at 127.9652 110.49 0)
 			(effects
@@
 			)
 		)
-		(property "Footprint" "PCM_Resistor_SMD_AKL:R_0603_1608Metric"
+		(property "Footprint" "Resistor_SMD:R_0603_1608Metric"
 			(at 123.698 116.84 90)
 			(effects
@@
 			)
 		)
-		(property "Footprint" "PCM_Capacitor_SMD_AKL:C_0805_2012Metric"
+		(property "Footprint" "Capacitor_SMD:C_0805_2012Metric"
 			(at 108.9152 102.87 0)
 			(effects
@@
 			)
 		)
-		(property "Footprint" "PCM_Resistor_SMD_AKL:R_0402_1005Metric"
+		(property "Footprint" "Resistor_SMD:R_0402_1005Metric"
 			(at 222.25 113.03 0)
 			(effects
@@
 			)
 		)
-		(property "Footprint" "PCM_Resistor_SMD_AKL:R_0402_1005Metric"
+		(property "Footprint" "Resistor_SMD:R_0402_1005Metric"
 			(at 222.25 121.92 0)
 			(effects
@@
 			)
 		)
-		(property "Footprint" "PCM_Capacitor_SMD_AKL:C_1206_3216Metric"
+		(property "Footprint" "Capacitor_SMD:C_1206_3216Metric"
 			(at 117.8052 110.49 0)
 			(effects
@@
 			)
 		)
-		(property "Footprint" "PCM_Capacitor_SMD_AKL:C_1206_3216Metric"
+		(property "Footprint" "Capacitor_SMD:C_1206_3216Metric"
 			(at 85.3948 110.49 0)
 			(effects
@@
 			)
 		)
-		(property "Footprint" "PCM_Capacitor_SMD_AKL:C_1206_3216Metric"
+		(property "Footprint" "Capacitor_SMD:C_1206_3216Metric"
 			(at 157.1752 110.49 0)
 			(effects
@@
 			)
 		)
-		(property "Footprint" "PCM_Capacitor_SMD_AKL:C_0805_2012Metric"
+		(property "Footprint" "Capacitor_SMD:C_0805_2012Metric"
 			(at 242.8748 115.57 0)
 			(effects
@@
 			)
 		)
-		(property "Footprint" "PCM_Capacitor_SMD_AKL:C_0603_1608Metric"
+		(property "Footprint" "Capacitor_SMD:C_0603_1608Metric"
 			(at 170.18 114.3 0)
 			(effects
@@
 			)
 		)
-		(property "Footprint" "PCM_Capacitor_SMD_AKL:C_0805_2012Metric"
+		(property "Footprint" "Capacitor_SMD:C_0805_2012Metric"
 			(at 251.1552 115.57 0)
 			(effects
@@
 			)
 		)
-		(property "Footprint" "PCM_Package_TO_SOT_SMD_AKL:SOT-23-6"
+		(property "Footprint" "Package_TO_SOT_SMD:SOT-23-6"
 			(at 164.846 95.758 0)
 			(effects
@@
 			)
 		)
-		(property "Footprint" "PCM_Capacitor_SMD_AKL:C_0402_1005Metric"
+		(property "Footprint" "Capacitor_SMD:C_0402_1005Metric"
 			(at 200.66 99.06 0)
 			(effects

Commit message: Bump versions
Parts:
- renumbered J703 to J701, J701 to J702, J702 to J703
Connections:
- net VIN renamed VIN_BUCK
Other:
- note removed: "Converter IC voltage range 4.5-50V, however, Vin needs to be a bit higher to give some headroom for the PTC fuse."
Changed lines of the file:
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@@
 	(title_block
 		(title "Hat Labs Serial Interface Device (HALSER)")
-		(date "2024-11-20")
-		(rev "1.0.0-a1")
+		(date "2024-12-20")
+		(rev "1.0.0")
 		(company "Hat Labs oy")
 		(comment 1 "https://creativecommons.org/licenses/by-sa/4.0")
@@
 		(stroke
 			(width 0)
-			(type default)
+			(type dash)
 		)
 	)
@@
 		(stroke
 			(width 0)
-			(type default)
+			(type dash)
 		)
 	)
@@
 		(stroke
 			(width 0)
-			(type default)
+			(type dash)
 		)
 	)
@@
 		(stroke
 			(width 0)
-			(type default)
+			(type dash)
 		)
 	)
@@
 		)
 	)
-	(text "Converter IC voltage range 4.5-50V,\nhowever, Vin needs to be a bit higher\nto give some headroom for the PTC\nfuse."
-		(exclude_from_sim no)
-		(at 180.848 85.344 0)
-		(effects
-			(font
-				(size 1.27 1.27)
-			)
-			(justify left bottom)
-		)
-	)
 	(text "Prevent feeding Vin to USB"
 		(exclude_from_sim no)
@@
 		)
 	)
-	(label "VIN"
+	(label "VIN_BUCK"
 		(at 146.05 102.87 0)
 		(fields_autoplaced yes)
@@
 		)
 	)
-	(label "Vin"
-		(at 58.42 53.34 0)
-		(fields_autoplaced yes)
-		(effects
-			(font
-				(size 1.27 1.27)
-			)
-			(justify left bottom)
-		)
-	)
 	(label "SW"
 		(at 198.12 107.95 180)
@@
 		(on_board yes)
 		(dnp no)
-		(property "Reference" "#PWR0706"
+		(property "Reference" "#PWR0707"
 			(at 156.21 116.84 0)
 			(effects
@@
 			(project "SH-ESP32"
 				(path "/dff502f1-2fe5-4c09-a767-aabc78c2e052/00000000-0000-0000-0000-00005f6faf6e"
-					(reference "#PWR0706")
+					(reference "#PWR0707")
 					(unit 1)
 				)
@@
 		(on_board yes)
 		(dnp no)
-		(property "Reference" "#PWR0711"
+		(property "Reference" "#PWR0712"
 			(at 250.19 121.92 0)
 			(effects
@@
 			(project "SH-ESP32"
 				(path "/dff502f1-2fe5-4c09-a767-aabc78c2e052/00000000-0000-0000-0000-00005f6faf6e"
-					(reference "#PWR0711")
+					(reference "#PWR0712")
 					(unit 1)
 				)
@@
 		(on_board yes)
 		(dnp no)
-		(property "Reference" "#PWR0708"
+		(property "Reference" "#PWR0709"
 			(at 185.42 128.27 0)
 			(effects
@@
 			(project "SH-ESP32"
 				(path "/dff502f1-2fe5-4c09-a767-aabc78c2e052/00000000-0000-0000-0000-00005f6faf6e"
-					(reference "#PWR0708")
+					(reference "#PWR0709")
 					(unit 1)
 				)
@@
 		(on_board yes)
 		(dnp no)
-		(property "Reference" "#PWR0712"
+		(property "Reference" "#PWR0713"
 			(at 261.62 111.76 0)
 			(effects
@@
 			(project "SH-ESP32"
 				(path "/dff502f1-2fe5-4c09-a767-aabc78c2e052/00000000-0000-0000-0000-00005f6faf6e"
-					(reference "#PWR0712")
+					(reference "#PWR0713")
 					(unit 1)
 				)
@@
 		(on_board yes)
 		(dnp no)
-		(property "Reference" "J701"
+		(property "Reference" "J702"
 			(at 44.196 44.704 0)
 			(effects
@@
 			(project "SH-ESP32"
 				(path "/dff502f1-2fe5-4c09-a767-aabc78c2e052/00000000-0000-0000-0000-00005f6faf6e"
-					(reference "J701")
+					(reference "J702")
 					(unit 1)
 				)
@@
 		(on_board yes)
 		(dnp no)
-		(property "Reference" "#PWR0709"
+		(property "Reference" "#PWR0710"
 			(at 222.25 133.35 0)
 			(effects
@@
 			(project "SH-ESP32"
 				(path "/dff502f1-2fe5-4c09-a767-aabc78c2e052/00000000-0000-0000-0000-00005f6faf6e"
-					(reference "#PWR0709")
+					(reference "#PWR0710")
 					(unit 1)
 				)
@@
 		(dnp no)
 		(fields_autoplaced yes)
-		(property "Reference" "#PWR0713"
+		(property "Reference" "#PWR0706"
 			(at 149.86 147.32 0)
 			(effects
@@
 			(project ""
 				(path "/dff502f1-2fe5-4c09-a767-aabc78c2e052/00000000-0000-0000-0000-00005f6faf6e"
-					(reference "#PWR0713")
+					(reference "#PWR0706")
 					(unit 1)
 				)
@@
 		(on_board yes)
 		(dnp no)
-		(property "Reference" "#PWR0710"
+		(property "Reference" "#PWR0711"
 			(at 243.84 121.92 0)
 			(effects
@@
 			(project "SH-ESP32"
 				(path "/dff502f1-2fe5-4c09-a767-aabc78c2e052/00000000-0000-0000-0000-00005f6faf6e"
-					(reference "#PWR0710")
+					(reference "#PWR0711")
 					(unit 1)
 				)
@@
 		(on_board yes)
 		(dnp no)
-		(property "Reference" "#PWR0707"
+		(property "Reference" "#PWR0708"
 			(at 170.18 125.73 0)
 			(effects
@@
 			(project "SH-ESP32"
 				(path "/dff502f1-2fe5-4c09-a767-aabc78c2e052/00000000-0000-0000-0000-00005f6faf6e"
-					(reference "#PWR0707")
+					(reference "#PWR0708")
 					(unit 1)
 				)
@@
 		(dnp no)
 		(fields_autoplaced yes)
-		(property "Reference" "J702"
+		(property "Reference" "J703"
 			(at 157.48 128.27 0)
 			(effects
@@
 			(project ""
 				(path "/dff502f1-2fe5-4c09-a767-aabc78c2e052/00000000-0000-0000-0000-00005f6faf6e"
-					(reference "J702")
+					(reference "J703")
 					(unit 1)
 				)
@@
 		(on_board yes)
 		(dnp no)
-		(property "Reference" "J703"
+		(property "Reference" "J701"
 			(at 44.196 25.654 0)
 			(effects
@@
 			(project "HALSER"
 				(path "/dff502f1-2fe5-4c09-a767-aabc78c2e052/00000000-0000-0000-0000-00005f6faf6e"
-					(reference "J703")
+					(reference "J701")
 					(unit 1)
 				)
